Commit message: Fix some errors

File: urdf/world/world.urdf.xacro (robot description, xacro)
@@ -8,10 +8,10 @@
     <visual>
       <geometry>
-        <mesh filename="package://mrover/urdf/meshes/ground_boulders.fbx"/>
+        <mesh filename="package://mrover/urdf/meshes/ground.fbx"/>
       </geometry>
     </visual>
     <collision>
       <geometry>
-        <mesh filename="package://mrover/urdf/meshes/ground_boulders.fbx"/>
+        <mesh filename="package://mrover/urdf/meshes/ground.fbx"/>
       </geometry>
     </collision>

Commit message: add sim flat world

File: urdf/world/world.urdf.xacro (robot description, xacro)
@@ -8,10 +8,10 @@
     <visual>
       <geometry>
-        <mesh filename="package://mrover/urdf/meshes/ground.fbx"/>
+        <mesh filename="package://mrover/urdf/meshes/groundflat.fbx"/>
       </geometry>
     </visual>
     <collision>
       <geometry>
-        <mesh filename="package://mrover/urdf/meshes/ground.fbx"/>
+        <mesh filename="package://mrover/urdf/meshes/groundflat.fbx"/>
       </geometry>
     </collision>

Commit message: Better ground

File: urdf/world/world.urdf.xacro (robot description, xacro)
@@ -8,10 +8,10 @@
     <visual>
       <geometry>
-        <mesh filename="package://mrover/urdf/meshes/groundflat.fbx"/>
+        <mesh filename="package://mrover/urdf/meshes/TexturedGround.fbx"/>
       </geometry>
     </visual>
     <collision>
       <geometry>
-        <mesh filename="package://mrover/urdf/meshes/groundflat.fbx"/>
+        <mesh filename="package://mrover/urdf/meshes/TexturedGround.fbx"/>
       </geometry>
     </collision>

Commit message: idk

File: urdf/world/world.urdf.xacro (robot description, xacro)
@@ -8,10 +8,10 @@
     <visual>
       <geometry>
-        <mesh filename="package://mrover/urdf/meshes/textured_ground.fbx"/>
+        <mesh filename="package://mrover/urdf/meshes/groundflat.fbx"/>
       </geometry>
     </visual>
     <collision>
       <geometry>
-        <mesh filename="package://mrover/urdf/meshes/textured_ground_decimated.fbx"/>
+        <mesh filename="package://mrover/urdf/meshes/groundflat.fbx"/>
       </geometry>
     </collision>

Commit message: pre normal based filtering

File: urdf/world/world.urdf.xacro (robot description, xacro)
@@ -8,10 +8,10 @@
     <visual>
       <geometry>
-        <mesh filename="package://mrover/urdf/meshes/groundflat.fbx"/>
+        <mesh filename="package://mrover/urdf/meshes/textured_ground.fbx"/>
       </geometry>
     </visual>
     <collision>
       <geometry>
-        <mesh filename="package://mrover/urdf/meshes/groundflat.fbx"/>
+        <mesh filename="package://mrover/urdf/meshes/textured_ground_decimated.fbx"/>
       </geometry>
     </collision>

Commit message: new terrain

File: urdf/world/world.urdf.xacro (robot description, xacro)
@@ -8,10 +8,10 @@
     <visual>
       <geometry>
-        <mesh filename="package://mrover/urdf/meshes/groundflat.fbx"/>
+        <mesh filename="package://mrover/urdf/meshes/mars-sol-239.fbx"/>
       </geometry>
     </visual>
     <collision>
       <geometry>
-        <mesh filename="package://mrover/urdf/meshes/groundflat.fbx"/>
+        <mesh filename="package://mrover/urdf/meshes/mars-sol-239-decimated.fbx"/>
       </geometry>
     </collision>

Commit message: found eigen vectors and values

File: urdf/world/world.urdf.xacro (robot description, xacro)
@@ -8,10 +8,10 @@
     <visual>
       <geometry>
-        <mesh filename="package://mrover/urdf/meshes/groundflat.fbx"/>
+        <mesh filename="package://mrover/urdf/meshes/ground.fbx"/>
       </geometry>
     </visual>
     <collision>
       <geometry>
-        <mesh filename="package://mrover/urdf/meshes/groundflat.fbx"/>
+        <mesh filename="package://mrover/urdf/meshes/ground.fbx"/>
       </geometry>
     </collision>
