Commit message: Committing Pure Pursuit

File: urdf/world/small_rock.urdf.xacro (robot description, xacro)
@@ -1,11 +1,11 @@
 <?xml version="1.0"?>
 <robot xmlns:xacro="http://www.ros.org/wiki/xacro" name="rover">
-  <xacro:property name="mass" value="1.36078"/>\
+  <xacro:property name="mass" value="0"/><!--1.36078-->
   <link name="base_link">
     <inertial>
       <mass value="${mass}"/>
-      <inertia ixx="0.01" ixy="0" ixz="0"
-               iyy="0.01" iyz="0"
-               izz="0.01"/>
+      <inertia ixx="0" ixy="0" ixz="0"
+               iyy="0" iyz="0"
+               izz="0"/>
     </inertial>
     <visual>
