Commit message: bruh

File: urdf/world/lander.urdf.xacro (robot description, xacro)
@@ -13,5 +13,5 @@
     <collision>
       <geometry>
-        <mesh filename="package://mrover/urdf/meshes/lander.fbx" />
+        <mesh filename="package://mrover/urdf/meshes/lander_and_keyboard.fbx" />
       </geometry>
     </collision>

Commit message: auto typing sequence with presses

File: urdf/world/lander.urdf.xacro (robot description, xacro)
@@ -13,5 +13,5 @@
     <collision>
       <geometry>
-        <mesh filename="package://mrover/urdf/meshes/lander_and_keyboard.fbx" />
+        <mesh filename="package://mrover/urdf/meshes/lander_and_keyboard_small.fbx" />
       </geometry>
     </collision>

Commit message: better lander

File: urdf/world/lander.urdf.xacro (robot description, xacro)
@@ -13,5 +13,5 @@
     <collision>
       <geometry>
-        <mesh filename="package://mrover/urdf/meshes/lander.fbx" />
+        <mesh filename="package://mrover/urdf/meshes/lander_and_keyboard_small.fbx" />
       </geometry>
     </collision>

Commit message: better lander stuff

File: urdf/world/lander.urdf.xacro (robot description, xacro)
@@ -8,5 +8,5 @@
     <visual>
       <geometry>
-        <mesh filename="package://mrover/urdf/meshes/lander_and_keyboard.fbx" />
+        <mesh filename="package://mrover/urdf/meshes/lander_and_keyboard_small.fbx" />
       </geometry>
     </visual>

Commit message: better filming

File: urdf/world/lander.urdf.xacro (robot description, xacro)
@@ -13,5 +13,5 @@
     <collision>
       <geometry>
-        <mesh filename="package://mrover/urdf/meshes/lander_and_keyboard_small.fbx" />
+        <mesh filename="package://mrover/urdf/meshes/rock.fbx"/>
       </geometry>
     </collision>

Commit message: decimate lander

File: urdf/world/lander.urdf.xacro (robot description, xacro)
@@ -13,5 +13,5 @@
     <collision>
       <geometry>
-        <mesh filename="package://mrover/urdf/meshes/lander.fbx"/>
+        <mesh filename="package://mrover/urdf/meshes/lander_decimated.fbx"/>
       </geometry>
     </collision>

Commit message: Co-authored-by: Calvin <eternaks@users.noreply.github.com>

File: urdf/world/lander.urdf.xacro (robot description, xacro)
@@ -3,6 +3,6 @@
   <link name="base_link">
     <inertial>
-      <mass value="100" />
-      <inertia ixx="10" ixy="10" ixz="10" iyy="10" iyz="10" izz="10" />
+      <mass value="0" />
+      <inertia ixx="0" ixy="0" ixz="0" iyy="0" iyz="0" izz="0" />
     </inertial>
     <visual>
