Commit message: better physics meshes

File: urdf/world/large_rock.urdf.xacro (robot description, xacro)
@@ -16,5 +16,5 @@
     <collision>
       <geometry>
-        <mesh filename="package://mrover/urdf/meshes/large_rock.fbx"/>
+        <mesh filename="package://mrover/urdf/meshes/large_rock_decimated.fbx"/>
       </geometry>
     </collision>

File: urdf/world/medium_rock.urdf.xacro (robot description, xacro)
@@ -16,5 +16,5 @@
     <collision>
       <geometry>
-        <mesh filename="package://mrover/urdf/meshes/medium_rock.fbx"/>
+        <mesh filename="package://mrover/urdf/meshes/medium_rock_decimated.fbx"/>
       </geometry>
     </collision>

File: urdf/world/small_rock.urdf.xacro (robot description, xacro)
@@ -16,5 +16,5 @@
     <collision>
       <geometry>
-        <mesh filename="package://mrover/urdf/meshes/small_rock.fbx"/>
+        <mesh filename="package://mrover/urdf/meshes/small_rock_decimated.fbx"/>
       </geometry>
     </collision>

File: urdf/world/world.urdf.xacro (robot description, xacro)
@@ -8,10 +8,10 @@
     <visual>
       <geometry>
-        <mesh filename="package://mrover/urdf/meshes/TexturedGround.fbx"/>
+        <mesh filename="package://mrover/urdf/meshes/textured_ground.fbx"/>
       </geometry>
     </visual>
     <collision>
       <geometry>
-        <mesh filename="package://mrover/urdf/meshes/TexturedGround.fbx"/>
+        <mesh filename="package://mrover/urdf/meshes/textured_ground_decimated.fbx"/>
       </geometry>
     </collision>

Commit message: Simulator changes to prevent fake high cost and make good SAR videos

File: urdf/world/large_rock.urdf.xacro (robot description, xacro)
@@ -1,11 +1,11 @@
 <?xml version="1.0"?>
 <robot xmlns:xacro="http://www.ros.org/wiki/xacro" name="rover">
-  <xacro:property name="mass" value="1.36078"/>\
+  <xacro:property name="mass" value="0"/>\
   <link name="base_link">
     <inertial>
       <mass value="${mass}"/>
-      <inertia ixx="0.01" ixy="0" ixz="0"
-               iyy="0.01" iyz="0"
-               izz="0.01"/>
+      <inertia ixx="0" ixy="0" ixz="0"
+               iyy="0" iyz="0"
+               izz="0"/>
     </inertial>
     <visual>
