Commit message: added new gripped 3d files, full rover assembled

File: urdf/rover/rover.urdf (robot description, URDF)
Before this commit: robot rover, 25 links, 11 joints
Links:
- removed link arm_gripper_link
- link arm_a_link: mass None -> 1; geometry collision box size=0.085 0.1 0.1; visual mesh filename=package://mrover/urdf/meshes/arm_a.fbx
- link arm_b_link: mass None -> 1; geometry collision box size=0.49299999999999994 0.04 0.04; visual mesh filename=package://mrover/urdf/meshes/arm_b.fbx
- link arm_base_link: mass 3.0 -> None; geometry 
- link arm_c_link: mass None -> 1; geometry collision box size=0.4675 0.04 0.04; visual mesh filename=package://mrover/urdf/meshes/arm_c.fbx
- link arm_d_link: mass None -> 1; geometry collision box size=0.05525 0.15 0.065; visual mesh filename=package://mrover/urdf/meshes/arm_d.fbx
- link arm_e_link: mass None -> 1; geometry collision box size=0.1275 0.155 0.032; visual mesh filename=package://mrover/urdf/meshes/arm_e.fbx
- link back_left_wheel_link: geometry collision cylinder length=0.08 radius=0.13; visual mesh filename=package://mrover/urdf/meshes/rover_left_wheel.fbx
- link back_right_wheel_link: geometry collision cylinder length=0.08 radius=0.13; visual mesh filename=package://mrover/urdf/meshes/rover_right_wheel.fbx
- link center_left_wheel_link: geometry collision cylinder length=0.08 radius=0.13; visual mesh filename=package://mrover/urdf/meshes/rover_left_wheel.fbx
- link center_right_wheel_link: geometry collision cylinder length=0.08 radius=0.13; visual mesh filename=package://mrover/urdf/meshes/rover_right_wheel.fbx
- link chassis_link: geometry collision box size=0.167 0.63 0.0891; collision box size=0.277 0.63 0.183
- link front_left_wheel_link: geometry collision cylinder length=0.08 radius=0.13; visual mesh filename=package://mrover/urdf/meshes/rover_left_wheel.fbx
- link front_right_wheel_link: geometry collision cylinder length=0.08 radius=0.13; visual mesh filename=package://mrover/urdf/meshes/rover_right_wheel.fbx
- link left_bogie_link: geometry collision box size=0.2 0.025 0.025; collision box size=0.2 0.025 0.025
- link left_rocker_link: geometry collision box size=0.2 0.025 0.025; collision box size=0.5 0.025 0.025
- link right_bogie_link: geometry collision box size=0.2 0.025 0.025; collision box size=0.2 0.025 0.025
- link right_rocker_link: geometry collision box size=0.2 0.025 0.025; collision box size=0.5 0.025 0.025
Joints:
- removed joint arm_a_to_arm_b
- removed joint arm_b_to_arm_c
- removed joint arm_c_to_arm_d
- removed joint arm_d_to_arm_e
- removed joint chassis_to_arm_a
- removed joint gripper_link
- added joint arm_a_link_to_arm_b_link: type revolute, parent arm_a_link, child arm_b_link, origin xyz=0.034346 0 0.049024, axis 0 1 0, limit lower=-0.7853981875 upper=0 effort=0 velocity=0
- added joint arm_b_link_to_arm_c_link: type revolute, parent arm_b_link, child arm_c_link, origin xyz=0.534365 0 0.009056, axis 0 1 0, limit lower=-0.959931 upper=2.87979 effort=0 velocity=0
- added joint arm_c_link_to_arm_d_link: type revolute, parent arm_c_link, child arm_d_link, origin xyz=0.546033 0 0.088594, axis 0 1 0, limit lower=-2.35619 upper=2.35619 effort=0 velocity=0
- added joint arm_d_link_to_arm_e_link: type revolute, parent arm_d_link, child arm_e_link, origin xyz=0.044886 0 0, axis 1 0 0, limit lower=-2.35619 upper=2.35619 effort=0 velocity=0
- added joint base_link_to_arm_base_link: type fixed, parent base_link, child arm_base_link, origin xyz=0.199228 -0.200235 0.540196
- added joint base_link_to_chassis_link: type fixed, parent base_link, child chassis_link, origin xyz=0 0 0.439675
- added joint chassis_link_to_arm_a_link: type prismatic, parent chassis_link, child arm_a_link, origin xyz=0.164882 -0.200235 0.051497, axis 0 1 0, limit lower=0 upper=0.4 effort=0 velocity=0
- added joint chassis_link_to_left_gps: type fixed, parent chassis_link, child left_gps, origin xyz=0 0.1 0
- added joint chassis_link_to_left_rocker_link: type revolute, parent chassis_link, child left_rocker_link, origin xyz=0.164665 0.365 0 rpy=-1.570796375 0 0, axis 0 0 1, limit lower=-0.122173 upper=0.523599 effort=0 velocity=0
- added joint chassis_link_to_right_rocker_link: type revolute, parent chassis_link, child right_rocker_link, origin xyz=0.164665 -0.365 0 rpy=-1.570796375 0 0, axis 0 0 1, limit lower=-0.122173 upper=0.523599 effort=0 velocity=0
- added joint left_bogie_link_to_center_left_wheel_link: type continuous, parent left_bogie_link, child center_left_wheel_link, origin xyz=-0.173532 0.147659 0.09, axis 0 0 1, limit effort=2.68 velocity=0
- added joint left_bogie_link_to_front_left_wheel_link: type continuous, parent left_bogie_link, child front_left_wheel_link, origin xyz=0.215233 0.147933 0.09, axis 0 0 1, limit effort=2.68 velocity=0
- added joint left_rocker_link_to_back_left_wheel_link: type continuous, parent left_rocker_link, child back_left_wheel_link, origin xyz=-0.417094 0.28513 0.09, axis 0 0 1, limit effort=2.68 velocity=0
- added joint left_rocker_link_to_left_bogie_link: type revolute, parent left_rocker_link, child left_bogie_link, origin xyz=0.198948 0.138674 0, axis 0 0 1, limit lower=-0.349066 upper=0.349066 effort=0 velocity=0
- added joint right_bogie_link_to_center_right_wheel_link: type continuous, parent right_bogie_link, child center_right_wheel_link, origin xyz=-0.173532 0.147659 -0.09, axis 0 0 1, limit effort=2.68 velocity=0
- added joint right_bogie_link_to_front_right_wheel_link: type continuous, parent right_bogie_link, child front_right_wheel_link, origin xyz=0.215233 0.147933 -0.09, axis 0 0 1, limit effort=2.68 velocity=0
- added joint right_rocker_link_to_back_right_wheel_link: type continuous, parent right_rocker_link, child back_right_wheel_link, origin xyz=-0.417094 0.28513 -0.09, axis 0 0 1, limit effort=2.68 velocity=0
- added joint right_rocker_link_to_right_bogie_link: type revolute, parent right_rocker_link, child right_bogie_link, origin xyz=0.198948 0.138674 0, axis 0 0 1, limit lower=-0.349066 upper=0.349066 effort=0 velocity=0
