Commit message: Rover driving in the sim :o

File: urdf/rover/rover.urdf.xacro (robot description, xacro)
@@ -63,5 +63,5 @@
   </xacro:macro>
   <xacro:macro name="wheel" params="pos side reflect">
-    <link name="${pos}_${side}_wheel_link">
+    <link name="${pos}_${side}">
       <xacro:cylinder_inertia m="${wheel_mass}" r="${wheel_radius}" h="${wheel_width}"/>
       <visual>
@@ -79,5 +79,5 @@
   <xacro:macro name="wheels" params="side reflect">
     <xacro:wheel pos="front" side="${side}" reflect="${reflect}"/>
-    <xacro:wheel pos="center" side="${side}" reflect="${reflect}"/>
+    <xacro:wheel pos="middle" side="${side}" reflect="${reflect}"/>
     <xacro:wheel pos="back" side="${side}" reflect="${reflect}"/>
     <link name="${side}_bogie_link">
@@ -128,7 +128,7 @@
       <limit lower="-0.122173" upper="0.523599" effort="0" velocity="0"/>
     </joint>
-    <joint name="${side}_rocker_link_to_back_${side}_wheel_link" type="continuous">
+    <joint name="${side}_rocker_link_to_back_${side}" type="continuous">
       <parent link="${side}_rocker_link"/>
-      <child link="back_${side}_wheel_link"/>
+      <child link="back_${side}"/>
       <origin xyz="-0.417094 0.28513 ${reflect * 0.09}"/>
       <axis xyz="0 0 1"/>
@@ -142,14 +142,14 @@
       <limit lower="-0.349066" upper="0.349066" effort="0" velocity="0"/>
     </joint>
-    <joint name="${side}_bogie_link_to_front_${side}_wheel_link" type="continuous">
+    <joint name="${side}_bogie_link_to_front_${side}" type="continuous">
       <parent link="${side}_bogie_link"/>
-      <child link="front_${side}_wheel_link"/>
+      <child link="front_${side}"/>
       <origin xyz="0.215233 0.147933 ${reflect * 0.09}"/>
       <axis xyz="0 0 1"/>
       <limit effort="${wheel_torque}" velocity="0"/>
     </joint>
-    <joint name="${side}_bogie_link_to_center_${side}_wheel_link" type="continuous">
+    <joint name="${side}_bogie_link_to_middle_${side}" type="continuous">
       <parent link="${side}_bogie_link"/>
-      <child link="center_${side}_wheel_link"/>
+      <child link="middle_${side}"/>
       <origin xyz="-0.173532 0.147659 ${reflect * 0.09}"/>
       <axis xyz="0 0 1"/>
@@ -232,10 +232,10 @@
   </joint>
   <link name="right_gps"/>
-    <joint name="chassis_link_to_center_gps" type="fixed">
-      <origin xyz="0 0 1"/>
-      <parent link="chassis_link"/>
-      <child link="center_gps"/>
-    </joint>
-    <link name="center_gps"/>
+  <joint name="chassis_link_to_center_gps" type="fixed">
+    <origin xyz="0 0 1"/>
+    <parent link="chassis_link"/>
+    <child link="center_gps"/>
+  </joint>
+  <link name="center_gps"/>
   <joint name="chassis_link_to_imu" type="fixed">
     <origin xyz="0 0 0"/>
@@ -269,18 +269,18 @@
     </collision>
   </link>
-  <joint name="chassis_link_to_mast_link" type="fixed">
-    <origin xyz="0.0505 -0.086 0.558"/>
-    <parent link="chassis_link"/>
-    <child link="mast_link"/>
-  </joint>
-  <link name="mast_link"/>
-  <joint name="mast_link_to_zed_mini_camera" type="continuous">
-    <origin xyz="0.05 0 0.0"/>
-    <parent link="mast_link"/>
-    <child link="zed_mini_camera"/>
-    <axis xyz="0 0 1"/>
-    <limit effort="2.68" velocity="0"/>
-  </joint>
-  <link name="zed_mini_camera"/>
-  <!--  <xacro:include filename="$(find mrover)/urdf/rover/rover_gazebo_plugins.urdf.xacro"/>-->
+  <!-- TODO(quintin): I removed this for now, feel free to add it back when needed -->
+  <!--  <joint name="chassis_link_to_mast_link" type="fixed">-->
+  <!--    <origin xyz="0.0505 -0.086 0.558"/>-->
+  <!--    <parent link="chassis_link"/>-->
+  <!--    <child link="mast_link"/>-->
+  <!--  </joint>-->
+  <!--  <link name="mast_link"/>-->
+  <!--  <joint name="mast_link_to_zed_mini_camera" type="continuous">-->
+  <!--    <origin xyz="0.05 0 0.0"/>-->
+  <!--    <parent link="mast_link"/>-->
+  <!--    <child link="zed_mini_camera"/>-->
+  <!--    <axis xyz="0 0 1"/>-->
+  <!--    <limit effort="2.68" velocity="0"/>-->
+  <!--  </joint>-->
+  <!--  <link name="zed_mini_camera"/>-->
 </robot>

Commit message: Arm chillikng too

File: urdf/rover/rover.urdf.xacro (robot description, xacro)
@@ -63,5 +63,5 @@
   </xacro:macro>
   <xacro:macro name="wheel" params="pos side reflect">
-    <link name="${pos}_${side}">
+    <link name="${pos}_${side}_wheel_link">
       <xacro:cylinder_inertia m="${wheel_mass}" r="${wheel_radius}" h="${wheel_width}"/>
       <visual>
@@ -79,5 +79,5 @@
   <xacro:macro name="wheels" params="side reflect">
     <xacro:wheel pos="front" side="${side}" reflect="${reflect}"/>
-    <xacro:wheel pos="middle" side="${side}" reflect="${reflect}"/>
+    <xacro:wheel pos="center" side="${side}" reflect="${reflect}"/>
     <xacro:wheel pos="back" side="${side}" reflect="${reflect}"/>
     <link name="${side}_bogie_link">
@@ -128,7 +128,7 @@
       <limit lower="-0.122173" upper="0.523599" effort="0" velocity="0"/>
     </joint>
-    <joint name="${side}_rocker_link_to_back_${side}" type="continuous">
+    <joint name="${side}_rocker_link_to_back_${side}_wheel_link" type="continuous">
       <parent link="${side}_rocker_link"/>
-      <child link="back_${side}"/>
+      <child link="back_${side}_wheel_link"/>
       <origin xyz="-0.417094 0.28513 ${reflect * 0.09}"/>
       <axis xyz="0 0 1"/>
@@ -142,14 +142,14 @@
       <limit lower="-0.349066" upper="0.349066" effort="0" velocity="0"/>
     </joint>
-    <joint name="${side}_bogie_link_to_front_${side}" type="continuous">
+    <joint name="${side}_bogie_link_to_front_${side}_wheel_link" type="continuous">
       <parent link="${side}_bogie_link"/>
-      <child link="front_${side}"/>
+      <child link="front_${side}_wheel_link"/>
       <origin xyz="0.215233 0.147933 ${reflect * 0.09}"/>
       <axis xyz="0 0 1"/>
       <limit effort="${wheel_torque}" velocity="0"/>
     </joint>
-    <joint name="${side}_bogie_link_to_middle_${side}" type="continuous">
+    <joint name="${side}_bogie_link_to_center_${side}_wheel_link" type="continuous">
       <parent link="${side}_bogie_link"/>
-      <child link="middle_${side}"/>
+      <child link="center_${side}_wheel_link"/>
       <origin xyz="-0.173532 0.147659 ${reflect * 0.09}"/>
       <axis xyz="0 0 1"/>

Commit message: gripper working in sim

File: urdf/rover/rover.urdf.xacro (robot description, xacro)
@@ -195,4 +195,20 @@
   <xacro:arm_link name="d" m="1" x="0.065" y="0.15" z="0.065"/>
   <xacro:arm_link name="e" m="1" x="0.15" y="0.155" z="0.032"/>
+  <!-- TODO: figure out why this is cooked -->
+  <!-- <xacro:arm_link name="gripper" m="1" x="0.13" y="0.02" z="0.03"/> -->
+  <link name="arm_gripper_link">
+    <xacro:box_inertia m="1" d="0.02" w="0.13" h="0.03"/>
+    <visual>
+      <geometry>
+        <mesh filename="package://mrover/urdf/meshes/arm_gripper.fbx"/>
+      </geometry>
+    </visual>
+    <collision>
+      <origin xyz="$0.0875 0 0"/>
+      <geometry>
+        <box size="0.085 0.02 0.03"/>
+      </geometry>
+    </collision>
+  </link>
   <joint name="chassis_link_to_arm_a_link" type="prismatic">
     <origin xyz="0.164882 -0.200235 0.051497"/>
@@ -217,4 +233,11 @@
     <axis xyz="1 0 0"/>
     <limit lower="-2.35619" upper="2.35619" effort="0" velocity="0"/>
+  </joint>
+  <joint name="arm_e_link_to_arm_gripper_link" type="prismatic">
+    <origin xyz="0.0 0.079 0.0"/>
+    <parent link="arm_e_link"/>
+    <child link="arm_gripper_link"/>
+    <axis xyz="0 -1 0"/>
+    <limit lower="0" upper="0.08" effort="0" velocity="0"/>
   </joint>
   <xacro:wheels side="left" reflect="1"/>

Commit message: Add new rover model to sim

File: urdf/rover/rover.urdf.xacro (robot description, xacro)
@@ -2,5 +2,5 @@
 <robot xmlns:xacro="http://www.ros.org/wiki/xacro" name="rover">
   <!-- Constants -->
-  <xacro:property name="base_width" value="0.63"/>
+  <xacro:property name="base_width" value="0.635"/>
   <xacro:property name="base_len" value="0.478"/>
   <xacro:property name="base_height" value="0.183"/>
@@ -10,5 +10,19 @@
   <xacro:property name="chassis_mass" value="15"/>
   <xacro:property name="wheel_torque" value="2.68"/>
-  <xacro:property name="TAU" value="6.2831855"/>
+  <!-- Suspension link lengths (measured from blender) -->
+  <xacro:property name="rocker_front_length" value="0.44752"/>
+  <xacro:property name="rocker_front_angle" value="${39*pi/180}"/>
+  <xacro:property name="rocker_rear_length" value="0.281575"/>
+  <xacro:property name="rocker_rear_angle" value="${170*pi/180}"/>
+  <xacro:property name="double_lambda_base_length" value="0.14239"/>
+  <xacro:property name="double_lambda_base_angle" value="${pi/2}"/>
+  <xacro:property name="double_lambda_base_offset" value="-0.03810"/>
+  <xacro:property name="double_lambda_crank_length" value="0.09187"/>
+  <xacro:property name="double_lambda_crank_angle" value="${-39.603*pi/180}"/>
+  <xacro:property name="double_lambda_lower_length" value="0.16767"/>
+  <xacro:property name="double_lambda_lower_angle" value="${-20*pi/180}"/>
+  <xacro:property name="double_lambda_long_length" value="0.38313"/>
+  <xacro:property name="double_lambda_long_angle" value="${58.871*pi/180}"/>
+  <xacro:property name="double_lambda_long_shift" value="0.16767"/>
   <!-- Inertial Macros-->
   <xacro:macro name="cylinder_inertia" params="m r h">
@@ -77,28 +91,17 @@
     </link>
   </xacro:macro>
+  <!-- creates a collider that extends like a ray of some length at some angle (by default) -->
+  <xacro:macro name="suspension_collider" params="length width:=0.025 height:=0.025 angle dx:=0 dy:=0 dz:=0">
+    <collision>
+      <origin xyz="${length * cos(angle)/2 + dx} ${length * sin(angle)/2 + dy} ${dz}" rpy="0 0 ${angle}"/>
+      <geometry>
+        <box size="${length * 0.75} ${width} ${height}"/>
+      </geometry>
+    </collision>
+  </xacro:macro>
   <xacro:macro name="wheels" params="side reflect">
     <xacro:wheel pos="front" side="${side}" reflect="${reflect}"/>
     <xacro:wheel pos="center" side="${side}" reflect="${reflect}"/>
     <xacro:wheel pos="back" side="${side}" reflect="${reflect}"/>
-    <link name="${side}_bogie_link">
-      <xacro:box_inertia m="3" d="0.5" w="0.5" h="0.5"/>
-      <visual>
-        <geometry>
-          <mesh filename="package://mrover/urdf/meshes/rover_${side}_bogie.fbx"/>
-        </geometry>
-      </visual>
-      <collision>
-        <origin xyz="-0.14 0.1 0" rpy="0 0 -0.734"/>
-        <geometry>
-          <box size="0.2 0.025 0.025"/>
-        </geometry>
-      </collision>
-      <collision>
-        <origin xyz="0.1 0.088 0" rpy="0 0 0.734"/>
-        <geometry>
-          <box size="0.2 0.025 0.025"/>
-        </geometry>
-      </collision>
-    </link>
     <link name="${side}_rocker_link">
       <xacro:box_inertia m="3" d="0.5" w="0.5" h="0.5"/>
@@ -108,51 +111,142 @@
         </geometry>
       </visual>
-      <collision>
-        <origin xyz="0.11 0.077 0" rpy="0 0 0.585"/>
-        <geometry>
-          <box size="0.2 0.025 0.025"/>
-        </geometry>
-      </collision>
-      <collision>
-        <origin xyz="-0.22 0.15 0" rpy="0 0 -0.585"/>
-        <geometry>
-          <box size="0.5 0.025 0.025"/>
-        </geometry>
-      </collision>
+      <xacro:suspension_collider length="${rocker_front_length}" angle="${rocker_front_angle}"/>
+      <xacro:suspension_collider length="${rocker_rear_length}" angle="${rocker_rear_angle}"/>
+      <xacro:suspension_collider length="${double_lambda_base_length}" angle="${double_lambda_base_angle}"
+                                 dx="${rocker_rear_length * cos(rocker_rear_angle)}"
+                                 dy="${rocker_rear_length * sin(rocker_rear_angle) + double_lambda_base_offset}"/>
+    </link>
+    <link name="${side}_lambda_crank_rear_link">
+      <xacro:box_inertia m="3" d="0.1" w="0.1" h="0.1"/>
+      <visual>
+        <geometry>
+          <mesh filename="package://mrover/urdf/meshes/rover_rear_lambda_crank.fbx"/>
+        </geometry>
+      </visual>
+      <xacro:suspension_collider length="${double_lambda_crank_length}"
+                                 angle="${pi - double_lambda_crank_angle}"
+                                 height="0.008"/>
+    </link>
+    <link name="${side}_lambda_crank_front_link">
+      <xacro:box_inertia m="3" d="0.1" w="0.1" h="0.1"/>
+      <visual>
+        <geometry>
+          <mesh filename="package://mrover/urdf/meshes/rover_front_lambda_crank.fbx"/>
+        </geometry>
+      </visual>
+      <xacro:suspension_collider length="${double_lambda_crank_length}"
+                                 angle="${double_lambda_crank_angle}"
+                                 height="0.008"/>
+    </link>
+    <link name="${side}_lambda_lower_link">
+      <xacro:box_inertia m="2" d="0.5" w="0.5" h="0.5"/>
+      <visual>
+        <geometry>
+          <mesh filename="package://mrover/urdf/meshes/rover_${side}_lambda_lower.fbx"/>
+        </geometry>
+      </visual>
+      <xacro:suspension_collider length="${double_lambda_lower_length}" angle="${double_lambda_lower_angle}"/>
+      <xacro:suspension_collider length="${double_lambda_lower_length}" angle="${pi - double_lambda_lower_angle}"/>
+    </link>
+    <link name="${side}_lambda_front_link">
+      <xacro:box_inertia m="2" d="0.5" w="0.5" h="0.5"/>
+      <visual>
+        <geometry>
+          <mesh filename="package://mrover/urdf/meshes/rover_${side}_lambda_front.fbx"/>
+        </geometry>
+      </visual>
+      <xacro:suspension_collider length="${double_lambda_long_length}" angle="${double_lambda_long_angle}"
+                                 dx="${-double_lambda_long_shift * cos(double_lambda_long_angle)}"
+                                 dy="${-double_lambda_long_shift * sin(double_lambda_long_angle)}"/>
+    </link>
+    <link name="${side}_lambda_rear_link">
+      <xacro:box_inertia m="2" d="0.5" w="0.5" h="0.5"/>
+      <visual>
+        <geometry>
+          <mesh filename="package://mrover/urdf/meshes/rover_${side}_lambda_rear.fbx"/>
+        </geometry>
+      </visual>
+      <xacro:suspension_collider length="${double_lambda_long_length}" angle="${pi - double_lambda_long_angle}"
+                                 dx="${double_lambda_long_shift * cos(double_lambda_long_angle)}"
+                                 dy="${-double_lambda_long_shift * sin(double_lambda_long_angle)}"/>
     </link>
     <joint name="chassis_link_to_${side}_rocker_link" type="revolute">
       <parent link="chassis_link"/>
       <child link="${side}_rocker_link"/>
-      <origin xyz="0.164665 ${reflect * (base_width/2 + 0.05)} 0" rpy="${-TAU/4} 0 0"/>
+      <origin xyz="0.164665 ${reflect * (base_width/2 + 0.041)} 0" rpy="${-pi/2} 0 0"/>
       <axis xyz="0 0 1"/>
       <limit lower="-0.122173" upper="0.523599" effort="0" velocity="0"/>
     </joint>
-    <joint name="${side}_rocker_link_to_back_${side}_wheel_link" type="continuous">
+    <joint name="${side}_rocker_link_to_front_${side}_wheel_link" type="continuous">
       <parent link="${side}_rocker_link"/>
+      <child link="front_${side}_wheel_link"/>
+      <origin xyz="${rocker_front_length * cos(rocker_front_angle)}
+                   ${rocker_front_length * sin(rocker_front_angle)}
+                   ${reflect * 0.076}"/>
+      <axis xyz="0 0 1"/>
+      <limit effort="${wheel_torque}" velocity="0"/>
+    </joint>
+    <joint name="${side}_lambda_front_link_to_center_${side}_wheel_link" type="continuous">
+      <parent link="${side}_lambda_front_link"/>
+      <child link="center_${side}_wheel_link"/>
+      <origin xyz="${(double_lambda_long_length - double_lambda_long_shift) * cos(double_lambda_long_angle)}
+                   ${(double_lambda_long_length - double_lambda_long_shift) * sin(double_lambda_long_angle)}
+                   ${reflect * 0.076}"/>
+      <axis xyz="0 0 1"/>
+      <limit effort="${wheel_torque}" velocity="0"/>
+    </joint>
+    <joint name="${side}_lambda_rear_link_to_back_${side}_wheel_link" type="continuous">
+      <parent link="${side}_lambda_rear_link"/>
       <child link="back_${side}_wheel_link"/>
-      <origin xyz="-0.417094 0.28513 ${reflect * 0.09}"/>
+      <origin xyz="${-(double_lambda_long_length - double_lambda_long_shift) * cos(double_lambda_long_angle)}
+                   ${(double_lambda_long_length - double_lambda_long_shift) * sin(double_lambda_long_angle)}
+                   ${reflect * 0.076}"/>
       <axis xyz="0 0 1"/>
       <limit effort="${wheel_torque}" velocity="0"/>
     </joint>
-    <joint name="${side}_rocker_link_to_${side}_bogie_link" type="revolute">
+    <joint name="${side}_rocker_link_to_${side}_lambda_lower_link" type="continuous">
       <parent link="${side}_rocker_link"/>
-      <child link="${side}_bogie_link"/>
-      <origin xyz="0.198948 0.138674 0"/>
-      <axis xyz="0 0 1"/>
-      <limit lower="-0.349066" upper="0.349066" effort="0" velocity="0"/>
-    </joint>
-    <joint name="${side}_bogie_link_to_front_${side}_wheel_link" type="continuous">
-      <parent link="${side}_bogie_link"/>
-      <child link="front_${side}_wheel_link"/>
-      <origin xyz="0.215233 0.147933 ${reflect * 0.09}"/>
-      <axis xyz="0 0 1"/>
-      <limit effort="${wheel_torque}" velocity="0"/>
-    </joint>
-    <joint name="${side}_bogie_link_to_center_${side}_wheel_link" type="continuous">
-      <parent link="${side}_bogie_link"/>
-      <child link="center_${side}_wheel_link"/>
-      <origin xyz="-0.173532 0.147659 ${reflect * 0.09}"/>
-      <axis xyz="0 0 1"/>
-      <limit effort="${wheel_torque}" velocity="0"/>
+      <child link="${side}_lambda_lower_link"/>
+      <origin xyz="${rocker_rear_length * cos(rocker_rear_angle)}
+                   ${rocker_rear_length * sin(rocker_rear_angle) + double_lambda_base_offset + double_lambda_base_length}
+                   ${reflect * 0.045}"/>
+      <axis xyz="0 0 1"/>
+      <limit effort="0" velocity="0"/>
+    </joint>
+    <joint name="${side}_rocker_link_to_${side}_lambda_crank_front_link" type="revolute">
+      <parent link="${side}_rocker_link"/>
+      <child link="${side}_lambda_crank_front_link"/>
+      <origin xyz="${rocker_rear_length * cos(rocker_rear_angle)}
+                   ${rocker_rear_length * sin(rocker_rear_angle) + double_lambda_base_offset}
+                   ${reflect * 0.04}"/>
+      <axis xyz="0 0 1"/>
+      <limit upper="${-double_lambda_crank_angle}" lower="${-pi/2-double_lambda_crank_angle}" effort="0" velocity="0"/>
+    </joint>
+    <joint name="${side}_rocker_link_to_${side}_lambda_crank_rear_link" type="revolute">
+      <parent link="${side}_rocker_link"/>
+      <child link="${side}_lambda_crank_rear_link"/>
+      <origin xyz="${rocker_rear_length * cos(rocker_rear_angle)}
+                   ${rocker_rear_length * sin(rocker_rear_angle) + double_lambda_base_offset}
+                   ${reflect * 0.05}"/>
+      <axis xyz="0 0 1"/>
+      <limit upper="${pi/2+double_lambda_crank_angle}" lower="${double_lambda_crank_angle}" effort="0" velocity="0"/>
+    </joint>
+    <joint name="${side}_lambda_lower_link_to_${side}_lambda_front_link" type="continuous">
+      <parent link="${side}_lambda_lower_link"/>
+      <child link="${side}_lambda_front_link"/>
+      <origin xyz="${double_lambda_lower_length * cos(double_lambda_lower_angle)}
+                   ${double_lambda_lower_length * sin(double_lambda_lower_angle)}
+                   0"/>
+      <axis xyz="0 0 1"/>
+      <limit effort="0" velocity="0"/>
+    </joint>
+    <joint name="${side}_lambda_lower_link_to_${side}_lambda_rear_link" type="continuous">
+      <parent link="${side}_lambda_lower_link"/>
+      <child link="${side}_lambda_rear_link"/>
+      <origin xyz="${-double_lambda_lower_length * cos(double_lambda_lower_angle)}
+                   ${double_lambda_lower_length * sin(double_lambda_lower_angle)}
+                   0"/>
+      <axis xyz="0 0 1"/>
+      <limit effort="0" velocity="0"/>
     </joint>
   </xacro:macro>
@@ -167,5 +261,5 @@
     </visual>
     <collision>
-      <origin xyz="-0.085906 0 0"/>
+      <origin xyz="-0.085906 0 0.15"/>
       <geometry>
         <box size="0.277 ${base_width} ${base_height}"/>
@@ -173,5 +267,5 @@
     </collision>
     <collision>
-      <origin xyz="0.163609 0 -0.049449"/>
+      <origin xyz="0.163609 0 0"/>
       <geometry>
         <box size="0.167 ${base_width} 0.0891 "/>
@@ -204,5 +298,5 @@
   <xacro:arm_revolute_joint parent="arm_a" child="arm_b"
                             x="0.034346" y="0" z="0.049024"
-                            lower="${-TAU / 8}" upper="0"/>
+                            lower="${-pi / 8}" upper="0"/>
   <xacro:arm_revolute_joint parent="arm_b" child="arm_c"
                             x="0.534365" y="0" z="0.009056"

Commit message: camera in sim

File: urdf/rover/rover.urdf.xacro (robot description, xacro)
@@ -269,4 +269,10 @@
     </collision>
   </link>
+  <joint name="arm_e_link_to_finger_camera" type="fixed">
+    <origin xyz="0 0 0"/>
+    <parent link="arm_e_link"/>
+    <child link="finger_camera_frame"/>
+  </joint>
+  <link name="finger_camera_frame"/>
   <!-- TODO(quintin): I removed this for now, feel free to add it back when needed -->
   <!--  <joint name="chassis_link_to_mast_link" type="fixed">-->

Commit message: better camera angle

File: urdf/rover/rover.urdf.xacro (robot description, xacro)
@@ -270,6 +270,6 @@
   </link>
   <joint name="arm_e_link_to_finger_camera" type="fixed">
-    <origin xyz="0 0 0"/>
-    <parent link="arm_e_link"/>
+    <origin xyz="0 0 0" rpy="0 -${TAU/4} 0"/>
+    <parent link="arm_c_link"/>
     <child link="finger_camera_frame"/>
   </joint>

Commit message: moved camera back to join e

File: urdf/rover/rover.urdf.xacro (robot description, xacro)
@@ -293,6 +293,6 @@
   </link>
   <joint name="arm_e_link_to_finger_camera" type="fixed">
-    <origin xyz="0 0 0" rpy="0 -${TAU/4} 0"/>
-    <parent link="arm_c_link"/>
+    <origin xyz="0 0 0" rpy="0 0 0"/>
+    <parent link="arm_e_link"/>
     <child link="finger_camera_frame"/>
   </joint>

Commit message: moved camera back to join e

File: urdf/rover/rover.urdf.xacro (robot description, xacro)
@@ -270,6 +270,6 @@
   </link>
   <joint name="arm_e_link_to_finger_camera" type="fixed">
-    <origin xyz="0 0 0" rpy="0 -${TAU/4} 0"/>
-    <parent link="arm_c_link"/>
+    <origin xyz="0 0 0" rpy="0 0 0"/>
+    <parent link="arm_e_link"/>
     <child link="finger_camera_frame"/>
   </joint>
