Commit message: Add new sim map for testing the lander (#125)
* updated sim pathing

* Menu to select map

* prints the objects inside of the ytaml file

* loading from external yaml via yaml-cpp

* works in sim

* camera in sim

* test map

* added lander into the map

* style

* better camera angle

* urdf/textures/marker0.png: convert to Git LFS

* git lfs

* gitignore blend1 files

* correct sizing in blender

* moved camera back to join e

* reformatted input box

* remove unecessary

* remove ar tag generator

* removed IsDefined

* decimated

* updated the tags to have different ids on the lander

* style

* decimate lander

File: urdf/rover/rover.urdf.xacro (robot description, xacro)
@@ -292,4 +292,10 @@
     </collision>
   </link>
+  <joint name="arm_e_link_to_finger_camera" type="fixed">
+    <origin xyz="0 0 0" rpy="0 0 0"/>
+    <parent link="arm_e_link"/>
+    <child link="finger_camera_frame"/>
+  </joint>
+  <link name="finger_camera_frame"/>
   <!-- TODO(quintin): I removed this for now, feel free to add it back when needed -->
   <!--  <joint name="chassis_link_to_mast_link" type="fixed">-->

Commit message: Add new arm meshes + update urdf

File: urdf/rover/rover.urdf.xacro (robot description, xacro)
@@ -192,5 +192,5 @@
   <xacro:arm_link name="a" m="1" x="0.1" y="0.1" z="0.1"/>
   <xacro:arm_link name="b" m="1" x="0.58" y="0.04" z="0.04"/>
-  <xacro:arm_link name="c" m="1" x="0.55" y="0.04" z="0.04" dz="0.1"/>
+  <xacro:arm_link name="c" m="1" x="0.35" y="0.04" z="0.04" dz="0.1"/>
   <xacro:arm_link name="d" m="1" x="0.065" y="0.15" z="0.065"/>
   <xacro:arm_link name="e" m="1" x="0.15" y="0.155" z="0.032"/>
@@ -205,5 +205,5 @@
     </visual>
     <collision>
-      <origin xyz="$0.0875 0 0"/>
+      <origin xyz="0.0875 0 0"/>
       <geometry>
         <box size="0.085 0.02 0.03"/>
@@ -219,14 +219,14 @@
   </joint>
   <xacro:arm_revolute_joint parent="arm_a" child="arm_b"
-                            x="0.034346" y="0" z="0.049024"
-                            lower="${-TAU / 8}" upper="0"/>
+                            x="0.04452" y="0" z="0.05163"
+                            lower="-1.1344" upper="0.2617"/>
   <xacro:arm_revolute_joint parent="arm_b" child="arm_c"
-                            x="0.534365" y="0" z="0.009056"
-                            lower="-0.959931" upper="2.87979"/>
+                            x="0.53271" y="0" z="0"
+                            lower="-1.0471" upper="3.0543"/>
   <xacro:arm_revolute_joint parent="arm_c" child="arm_d"
-                            x="0.546033" y="0" z="0.088594"
-                            lower="-2.35619" upper="2.35619"/>
+                            x="0.39525" y="0" z="0.08329"
+                            lower="-1.1344" upper="1.1344"/>
   <joint name="arm_d_link_to_arm_e_link" type="revolute">
-    <origin xyz="0.044886 0 0"/>
+    <origin xyz="0 0 0"/>
     <parent link="arm_d_link"/>
     <child link="arm_e_link"/>
@@ -235,9 +235,9 @@
   </joint>
   <joint name="arm_e_link_to_arm_gripper_link" type="prismatic">
-    <origin xyz="0.0 0.079 0.0"/>
+    <origin xyz="0.08375 0.0 0.0"/>
     <parent link="arm_e_link"/>
     <child link="arm_gripper_link"/>
-    <axis xyz="0 -1 0"/>
-    <limit lower="0" upper="0.08" effort="0" velocity="0"/>
+    <axis xyz="0 1 0"/>
+    <limit lower="0" upper="0.088" effort="0" velocity="0"/>
   </joint>
   <xacro:wheels side="left" reflect="1"/>

Commit message: Add linear actuator to arm

File: urdf/rover/rover.urdf.xacro (robot description, xacro)
@@ -195,4 +195,6 @@
   <xacro:arm_link name="d" m="1" x="0.065" y="0.15" z="0.065"/>
   <xacro:arm_link name="e" m="1" x="0.15" y="0.155" z="0.032"/>
+  <xacro:arm_link name="la_base" m="0.1" x="0.01" y="0.01" z="0.08" dz="0.1"/>
+  <xacro:arm_link name="la_piston" m="0.1" x="0.01" y="0.01" z="0.05" dz="-0.05"/>
   <!-- TODO: figure out why this is cooked -->
   <!-- <xacro:arm_link name="gripper" m="1" x="0.13" y="0.02" z="0.03"/> -->
@@ -227,4 +229,7 @@
                             x="0.39525" y="0" z="0.08329"
                             lower="-1.1344" upper="1.1344"/>
+  <xacro:arm_revolute_joint parent="arm_a" child="arm_la_base"
+                            x="-0.00441" y="0" z="0.20149"
+                            lower="0" upper="2"/>
   <joint name="arm_d_link_to_arm_e_link" type="revolute">
     <origin xyz="0 0 0"/>
@@ -240,4 +245,11 @@
     <axis xyz="0 1 0"/>
     <limit lower="0" upper="0.088" effort="0" velocity="0"/>
+  </joint>
+  <joint name="arm_la_base_link_to_arm_la_piston_link" type="prismatic">
+    <origin xyz="0.0 0.0 0.32"/>
+    <parent link="arm_la_base_link"/>
+    <child link="arm_la_piston_link"/>
+    <axis xyz="0 0 1"/>
+    <limit lower="0" upper="0.25" effort="0" velocity="0"/>
   </joint>
   <xacro:wheels side="left" reflect="1"/>

Commit message: Update rover chassis

File: urdf/rover/rover.urdf.xacro (robot description, xacro)
@@ -124,5 +124,5 @@
       <parent link="chassis_link"/>
       <child link="${side}_rocker_link"/>
-      <origin xyz="0.164665 ${reflect * (base_width/2 + 0.05)} 0" rpy="${-TAU/4} 0 0"/>
+      <origin xyz="0.0 ${reflect * (base_width/2 + 0.05)} 0" rpy="${-TAU/4} 0 0"/>
       <axis xyz="0 0 1"/>
       <limit lower="-0.122173" upper="0.523599" effort="0" velocity="0"/>

Commit message: Add full suspension (a bit cooked)

File: urdf/rover/rover.urdf.xacro (robot description, xacro)
@@ -2,5 +2,5 @@
 <robot xmlns:xacro="http://www.ros.org/wiki/xacro" name="rover">
   <!-- Constants -->
-  <xacro:property name="base_width" value="0.63"/>
+  <xacro:property name="base_width" value="0.59892"/>
   <xacro:property name="base_len" value="0.478"/>
   <xacro:property name="base_height" value="0.183"/>
@@ -11,4 +11,20 @@
   <xacro:property name="wheel_torque" value="2.68"/>
   <xacro:property name="TAU" value="6.2831855"/>
+  <!-- Suspension link lengths (measured from blender) -->
+  <!-- TODO: make sure these are real for 2026 -->
+  <xacro:property name="rocker_front_length" value="0.44752"/>
+  <xacro:property name="rocker_front_angle" value="${39*pi/180}"/>
+  <xacro:property name="rocker_rear_length" value="0.281575"/>
+  <xacro:property name="rocker_rear_angle" value="${170*pi/180}"/>
+  <xacro:property name="double_lambda_base_length" value="0.14239"/>
+  <xacro:property name="double_lambda_base_angle" value="${pi/2}"/>
+  <xacro:property name="double_lambda_base_offset" value="-0.03810"/>
+  <xacro:property name="double_lambda_crank_length" value="0.09187"/>
+  <xacro:property name="double_lambda_crank_angle" value="${-39.603*pi/180}"/>
+  <xacro:property name="double_lambda_lower_length" value="0.16767"/>
+  <xacro:property name="double_lambda_lower_angle" value="${-20*pi/180}"/>
+  <xacro:property name="double_lambda_long_length" value="0.38313"/>
+  <xacro:property name="double_lambda_long_angle" value="${58.871*pi/180}"/>
+  <xacro:property name="double_lambda_long_shift" value="0.16767"/>
   <!-- Inertial Macros-->
   <xacro:macro name="cylinder_inertia" params="m r h">
@@ -77,28 +93,17 @@
     </link>
   </xacro:macro>
+  <!-- creates a collider that extends like a ray of some length at some angle (by default) -->
+  <xacro:macro name="suspension_collider" params="length width:=0.025 height:=0.025 angle dx:=0 dy:=0 dz:=0">
+    <collision>
+      <origin xyz="${length * cos(angle)/2 + dx} ${length * sin(angle)/2 + dy} ${dz}" rpy="0 0 ${angle}"/>
+      <geometry>
+        <box size="${length * 0.75} ${width} ${height}"/>
+      </geometry>
+    </collision>
+  </xacro:macro>
   <xacro:macro name="wheels" params="side reflect">
     <xacro:wheel pos="front" side="${side}" reflect="${reflect}"/>
     <xacro:wheel pos="center" side="${side}" reflect="${reflect}"/>
     <xacro:wheel pos="back" side="${side}" reflect="${reflect}"/>
-    <link name="${side}_bogie_link">
-      <xacro:box_inertia m="3" d="0.5" w="0.5" h="0.5"/>
-      <visual>
-        <geometry>
-          <mesh filename="package://mrover/urdf/meshes/rover_${side}_bogie.fbx"/>
-        </geometry>
-      </visual>
-      <collision>
-        <origin xyz="-0.14 0.1 0" rpy="0 0 -0.734"/>
-        <geometry>
-          <box size="0.2 0.025 0.025"/>
-        </geometry>
-      </collision>
-      <collision>
-        <origin xyz="0.1 0.088 0" rpy="0 0 0.734"/>
-        <geometry>
-          <box size="0.2 0.025 0.025"/>
-        </geometry>
-      </collision>
-    </link>
     <link name="${side}_rocker_link">
       <xacro:box_inertia m="3" d="0.5" w="0.5" h="0.5"/>
@@ -108,51 +113,128 @@
         </geometry>
       </visual>
-      <collision>
-        <origin xyz="0.11 0.077 0" rpy="0 0 0.585"/>
-        <geometry>
-          <box size="0.2 0.025 0.025"/>
-        </geometry>
-      </collision>
-      <collision>
-        <origin xyz="-0.22 0.15 0" rpy="0 0 -0.585"/>
-        <geometry>
-          <box size="0.5 0.025 0.025"/>
-        </geometry>
-      </collision>
+      <xacro:suspension_collider length="${rocker_front_length}" angle="${rocker_front_angle}" dz="${reflect * 0.06}"/>
+      <xacro:suspension_collider length="${rocker_rear_length}" angle="${rocker_rear_angle}" dz="${reflect * 0.06}"/>
+      <xacro:suspension_collider length="${double_lambda_base_length}" angle="${double_lambda_base_angle}"
+                                dx="${rocker_rear_length * cos(rocker_rear_angle)}"
+                                dy="${rocker_rear_length * sin(rocker_rear_angle) + double_lambda_base_offset}"
+                                dz="${reflect * 0.06}"/>
+    </link>
+    <link name="${side}_lambda_crank_rear_link">
+      <xacro:box_inertia m="3" d="0.1" w="0.1" h="0.1"/>
+      <visual>
+        <geometry>
+          <mesh filename="package://mrover/urdf/meshes/rover_rear_lambda_crank.fbx"/>
+        </geometry>
+      </visual>
+      <xacro:suspension_collider length="${double_lambda_crank_length}"
+                                 angle="${pi - double_lambda_crank_angle}"
+                                 height="0.008"/>
+    </link>
+    <link name="${side}_lambda_crank_front_link">
+      <xacro:box_inertia m="3" d="0.1" w="0.1" h="0.1"/>
+      <visual>
+        <geometry>
+          <mesh filename="package://mrover/urdf/meshes/rover_front_lambda_crank.fbx"/>
+        </geometry>
+      </visual>
+      <xacro:suspension_collider length="${double_lambda_crank_length}"
+                                 angle="${double_lambda_crank_angle}"
+                                 height="0.008"/>
+    </link>
+    <link name="${side}_lambda_lower_link">
+      <xacro:box_inertia m="2" d="0.5" w="0.5" h="0.5"/>
+      <visual>
+        <geometry>
+          <mesh filename="package://mrover/urdf/meshes/rover_${side}_lambda_lower.fbx"/>
+        </geometry>
+      </visual>
+      <xacro:suspension_collider length="${double_lambda_lower_length}" angle="${double_lambda_lower_angle}" dz="${reflect * 0.05}"/>
+      <xacro:suspension_collider length="${double_lambda_lower_length}" angle="${pi - double_lambda_lower_angle}" dz="${reflect * 0.05}"/>
+    </link>
+    <link name="${side}_lambda_front_link">
+      <xacro:box_inertia m="2" d="0.5" w="0.5" h="0.5"/>
+      <visual>
+        <geometry>
+          <mesh filename="package://mrover/urdf/meshes/rover_${side}_lambda_front.fbx"/>
+        </geometry>
+      </visual>
+      <xacro:suspension_collider length="${double_lambda_long_length}" angle="${double_lambda_long_angle}"
+                                 dx="${-double_lambda_long_shift * cos(double_lambda_long_angle)}"
+                                 dy="${-double_lambda_long_shift * sin(double_lambda_long_angle)}"/>
+    </link>
+    <link name="${side}_lambda_rear_link">
+      <xacro:box_inertia m="2" d="0.5" w="0.5" h="0.5"/>
+      <visual>
+        <geometry>
+          <mesh filename="package://mrover/urdf/meshes/rover_${side}_lambda_rear.fbx"/>
+        </geometry>
+      </visual>
+      <xacro:suspension_collider length="${double_lambda_long_length}" angle="${pi - double_lambda_long_angle}"
+                                 dx="${double_lambda_long_shift * cos(double_lambda_long_angle)}"
+                                 dy="${-double_lambda_long_shift * sin(double_lambda_long_angle)}"/>
     </link>
     <joint name="chassis_link_to_${side}_rocker_link" type="revolute">
       <parent link="chassis_link"/>
       <child link="${side}_rocker_link"/>
-      <origin xyz="0.0 ${reflect * (base_width/2 + 0.05)} 0" rpy="${-TAU/4} 0 0"/>
+      <origin xyz="0.0 ${reflect * (base_width/2)} 0" rpy="${-TAU/4} 0 0"/>
       <axis xyz="0 0 1"/>
       <limit lower="-0.122173" upper="0.523599" effort="0" velocity="0"/>
     </joint>
-    <joint name="${side}_rocker_link_to_back_${side}_wheel_link" type="continuous">
+    <joint name="${side}_rocker_link_to_front_${side}_wheel_link" type="continuous">
       <parent link="${side}_rocker_link"/>
+      <child link="front_${side}_wheel_link"/>
+      <origin xyz="0.34781 0.28303 ${reflect * 0.15200}"/>
+      <axis xyz="0 0 1"/>
+      <limit effort="${wheel_torque}" velocity="0"/>
+    </joint>
+    <joint name="${side}_lambda_front_link_to_center_${side}_wheel_link" type="continuous">
+      <parent link="${side}_lambda_front_link"/>
+      <child link="center_${side}_wheel_link"/>
+      <origin xyz="0.11343 0.18319 ${reflect * 0.09594}"/>
+      <axis xyz="0 0 1"/>
+      <limit effort="${wheel_torque}" velocity="0"/>
+    </joint>
+    <joint name="${side}_lambda_rear_link_to_back_${side}_wheel_link" type="continuous">
+      <parent link="${side}_lambda_rear_link"/>
       <child link="back_${side}_wheel_link"/>
-      <origin xyz="-0.417094 0.28513 ${reflect * 0.09}"/>
+      <origin xyz="-0.11343 0.18319 ${reflect * 0.09594}"/>
       <axis xyz="0 0 1"/>
       <limit effort="${wheel_torque}" velocity="0"/>
     </joint>
-    <joint name="${side}_rocker_link_to_${side}_bogie_link" type="revolute">
+    <joint name="${side}_rocker_link_to_${side}_lambda_lower_link" type="continuous">
       <parent link="${side}_rocker_link"/>
-      <child link="${side}_bogie_link"/>
-      <origin xyz="0.198948 0.138674 0"/>
-      <axis xyz="0 0 1"/>
-      <limit lower="-0.349066" upper="0.349066" effort="0" velocity="0"/>
-    </joint>
-    <joint name="${side}_bogie_link_to_front_${side}_wheel_link" type="continuous">
-      <parent link="${side}_bogie_link"/>
-      <child link="front_${side}_wheel_link"/>
-      <origin xyz="0.215233 0.147933 ${reflect * 0.09}"/>
-      <axis xyz="0 0 1"/>
-      <limit effort="${wheel_torque}" velocity="0"/>
-    </joint>
-    <joint name="${side}_bogie_link_to_center_${side}_wheel_link" type="continuous">
-      <parent link="${side}_bogie_link"/>
-      <child link="center_${side}_wheel_link"/>
-      <origin xyz="-0.173532 0.147659 ${reflect * 0.09}"/>
-      <axis xyz="0 0 1"/>
-      <limit effort="${wheel_torque}" velocity="0"/>
+      <child link="${side}_lambda_lower_link"/>
+      <!-- TODO: figure out what coordinate frame this is in -->
+      <origin xyz="-0.2773 0.15460 ${reflect * 0.05577}"/>
+      <axis xyz="0 0 1"/>
+      <limit effort="0" velocity="0"/>
+    </joint>
+    <joint name="${side}_rocker_link_to_${side}_lambda_crank_front_link" type="revolute">
+      <parent link="${side}_rocker_link"/>
+      <child link="${side}_lambda_crank_front_link"/>
+      <origin xyz="-0.27730 0.01220 ${reflect * 0.09809}"/>
+      <axis xyz="0 0 1"/>
+      <limit upper="${-double_lambda_crank_angle}" lower="${-pi/2-double_lambda_crank_angle}" effort="0" velocity="0"/>
+    </joint>
+    <joint name="${side}_rocker_link_to_${side}_lambda_crank_rear_link" type="revolute">
+      <parent link="${side}_rocker_link"/>
+      <child link="${side}_lambda_crank_rear_link"/>
+      <origin xyz="-0.27730 0.01220 ${reflect * 0.10760}"/>
+      <axis xyz="0 0 1"/>
+      <limit upper="${pi/2+double_lambda_crank_angle}" lower="${double_lambda_crank_angle}" effort="0" velocity="0"/>
+    </joint>
+    <joint name="${side}_lambda_lower_link_to_${side}_lambda_front_link" type="continuous">
+      <parent link="${side}_lambda_lower_link"/>
+      <child link="${side}_lambda_front_link"/>
+      <origin xyz="0.15755 -0.05735 ${reflect * 0.04708}"/>
+      <axis xyz="0 0 1"/>
+      <limit effort="0" velocity="0"/>
+    </joint>
+    <joint name="${side}_lambda_lower_link_to_${side}_lambda_rear_link" type="continuous">
+      <parent link="${side}_lambda_lower_link"/>
+      <child link="${side}_lambda_rear_link"/>
+      <origin xyz="-0.15755 -0.05735 ${reflect * 0.04708}"/>
+      <axis xyz="0 0 1"/>
+      <limit effort="0" velocity="0"/>
     </joint>
   </xacro:macro>
@@ -167,5 +249,5 @@
     </visual>
     <collision>
-      <origin xyz="-0.085906 0 0"/>
+      <origin xyz="-0.185906 0 0"/>
       <geometry>
         <box size="0.277 ${base_width} ${base_height}"/>
@@ -173,5 +255,5 @@
     </collision>
     <collision>
-      <origin xyz="0.163609 0 -0.049449"/>
+      <origin xyz="0.0 0 -0.049449"/>
       <geometry>
         <box size="0.167 ${base_width} 0.0891 "/>
@@ -180,4 +262,5 @@
   </link>
   <link name="arm_base_link"/>
+  <!-- TODO: recalculate -->
   <joint name="base_link_to_arm_base_link" type="fixed">
     <origin xyz="0.199228 -0.200235 0.540196"/>
@@ -214,5 +297,5 @@
   </link>
   <joint name="chassis_link_to_arm_a_link" type="prismatic">
-    <origin xyz="0.164882 -0.200235 0.051497"/>
+    <origin xyz="0.0 -0.200235 0.09870"/>
     <parent link="chassis_link"/>
     <child link="arm_a_link"/>
