Commit message: URDF tweaks

File: urdf/rover/rover.urdf.xacro (robot description, xacro)
@@ -5,26 +5,10 @@
   <xacro:property name="base_len" value="0.478"/>
   <xacro:property name="base_height" value="0.183"/>
-  <xacro:property name="wheel_radius" value="0.13"/>
-  <xacro:property name="wheel_width" value="0.08"/>
+  <xacro:property name="wheel_radius" value="0.12"/>
+  <xacro:property name="wheel_width" value="0.09"/>
   <xacro:property name="wheel_mass" value="3"/>
   <xacro:property name="chassis_mass" value="15"/>
   <xacro:property name="wheel_torque" value="2.68"/>
   <xacro:property name="TAU" value="6.2831855"/>
-  <!-- Suspension link lengths (measured from blender) -->
-  <!-- TODO: make sure these are real for 2026 -->
-  <xacro:property name="rocker_front_length" value="0.44752"/>
-  <xacro:property name="rocker_front_angle" value="${39*pi/180}"/>
-  <xacro:property name="rocker_rear_length" value="0.281575"/>
-  <xacro:property name="rocker_rear_angle" value="${170*pi/180}"/>
-  <xacro:property name="double_lambda_base_length" value="0.14239"/>
-  <xacro:property name="double_lambda_base_angle" value="${pi/2}"/>
-  <xacro:property name="double_lambda_base_offset" value="-0.03810"/>
-  <xacro:property name="double_lambda_crank_length" value="0.09187"/>
-  <xacro:property name="double_lambda_crank_angle" value="${-39.603*pi/180}"/>
-  <xacro:property name="double_lambda_lower_length" value="0.16767"/>
-  <xacro:property name="double_lambda_lower_angle" value="${-20*pi/180}"/>
-  <xacro:property name="double_lambda_long_length" value="0.38313"/>
-  <xacro:property name="double_lambda_long_angle" value="${58.871*pi/180}"/>
-  <xacro:property name="double_lambda_long_shift" value="0.16767"/>
   <!-- Inertial Macros-->
   <xacro:macro name="cylinder_inertia" params="m r h">
@@ -53,5 +37,5 @@
   </xacro:macro>
   <!-- Joints/Links Macros -->
-  <xacro:macro name="arm_link" params="name m x y z dz:=0">
+  <xacro:macro name="arm_link" params="name m x y z dx:=0 dz:=0">
     <link name="arm_${name}_link">
       <xacro:box_inertia m="${m}" d="${y}" w="${x}" h="${z}"/>
@@ -62,5 +46,5 @@
       </visual>
       <collision>
-        <origin xyz="${x / 2} 0 ${dz}"/>
+        <origin xyz="${x / 2 + dx} 0 ${dz}"/>
         <geometry>
           <box size="${x * 0.85} ${y} ${z}"/>
@@ -87,4 +71,5 @@
       </visual>
       <collision>
+      <origin xyz="0 0 ${reflect * -0.03}"/>
         <geometry>
           <cylinder length="${wheel_width}" radius="${wheel_radius}"/>
@@ -113,9 +98,9 @@
         </geometry>
       </visual>
-      <xacro:suspension_collider length="${rocker_front_length}" angle="${rocker_front_angle}" dz="${reflect * 0.06}"/>
-      <xacro:suspension_collider length="${rocker_rear_length}" angle="${rocker_rear_angle}" dz="${reflect * 0.06}"/>
-      <xacro:suspension_collider length="${double_lambda_base_length}" angle="${double_lambda_base_angle}"
-                                dx="${rocker_rear_length * cos(rocker_rear_angle)}"
-                                dy="${rocker_rear_length * sin(rocker_rear_angle) + double_lambda_base_offset}"
+      <xacro:suspension_collider length="0.44752" angle="0.68068" dz="${reflect * 0.06}"/>
+      <xacro:suspension_collider length="0.281575" angle="2.96706" dz="${reflect * 0.06}"/>
+      <xacro:suspension_collider length="0.14239" angle="${pi/2}"
+                                dx="-0.277297"
+                                dy="0.048894"
                                 dz="${reflect * 0.06}"/>
     </link>
@@ -127,6 +112,6 @@
         </geometry>
       </visual>
-      <xacro:suspension_collider length="${double_lambda_crank_length}"
-                                 angle="${pi - double_lambda_crank_angle}"
+      <xacro:suspension_collider length="0.09187"
+                                 angle="3.832795"
                                  height="0.008"/>
     </link>
@@ -138,6 +123,6 @@
         </geometry>
       </visual>
-      <xacro:suspension_collider length="${double_lambda_crank_length}"
-                                 angle="${double_lambda_crank_angle}"
+      <xacro:suspension_collider length="0.09187"
+                                 angle="-0.691203"
                                  height="0.008"/>
     </link>
@@ -149,6 +134,6 @@
         </geometry>
       </visual>
-      <xacro:suspension_collider length="${double_lambda_lower_length}" angle="${double_lambda_lower_angle}" dz="${reflect * 0.05}"/>
-      <xacro:suspension_collider length="${double_lambda_lower_length}" angle="${pi - double_lambda_lower_angle}" dz="${reflect * 0.05}"/>
+      <xacro:suspension_collider length="0.16767" angle="-0.349066" dz="${reflect * 0.05}"/>
+      <xacro:suspension_collider length="0.16767" angle="3.490659" dz="${reflect * 0.05}"/>
     </link>
     <link name="${side}_lambda_front_link">
@@ -159,7 +144,7 @@
         </geometry>
       </visual>
-      <xacro:suspension_collider length="${double_lambda_long_length}" angle="${double_lambda_long_angle}"
-                                 dx="${-double_lambda_long_shift * cos(double_lambda_long_angle)}"
-                                 dy="${-double_lambda_long_shift * sin(double_lambda_long_angle)}"/>
+      <xacro:suspension_collider length="0.38313" angle="1.027493"
+                                 dx="-0.086680"
+                                 dy="-0.143526"/>
     </link>
     <link name="${side}_lambda_rear_link">
@@ -170,7 +155,7 @@
         </geometry>
       </visual>
-      <xacro:suspension_collider length="${double_lambda_long_length}" angle="${pi - double_lambda_long_angle}"
-                                 dx="${double_lambda_long_shift * cos(double_lambda_long_angle)}"
-                                 dy="${-double_lambda_long_shift * sin(double_lambda_long_angle)}"/>
+      <xacro:suspension_collider length="0.38313" angle="2.114100"
+                                 dx="0.086680"
+                                 dy="-0.143526"/>
     </link>
     <joint name="chassis_link_to_${side}_rocker_link" type="revolute">
@@ -215,5 +200,5 @@
       <origin xyz="-0.27730 0.01220 ${reflect * 0.09809}"/>
       <axis xyz="0 0 1"/>
-      <limit upper="${-double_lambda_crank_angle}" lower="${-pi/2-double_lambda_crank_angle}" effort="0" velocity="0"/>
+      <limit upper="${pi/2}" lower="-${pi/2}" effort="0" velocity="0"/>
     </joint>
     <joint name="${side}_rocker_link_to_${side}_lambda_crank_rear_link" type="revolute">
@@ -222,5 +207,5 @@
       <origin xyz="-0.27730 0.01220 ${reflect * 0.10760}"/>
       <axis xyz="0 0 1"/>
-      <limit upper="${pi/2+double_lambda_crank_angle}" lower="${double_lambda_crank_angle}" effort="0" velocity="0"/>
+      <limit upper="${pi/2}" lower="-${pi/2}" effort="0" velocity="0"/>
     </joint>
     <joint name="${side}_lambda_lower_link_to_${side}_lambda_front_link" type="continuous">
@@ -273,9 +258,9 @@
     <child link="chassis_link"/>
   </joint>
-  <xacro:arm_link name="a" m="1" x="0.1" y="0.1" z="0.1"/>
+  <xacro:arm_link name="a" m="1" x="0.08" y="0.1" z="0.1"/>
   <xacro:arm_link name="b" m="1" x="0.58" y="0.04" z="0.04"/>
   <xacro:arm_link name="c" m="1" x="0.35" y="0.04" z="0.04" dz="0.1"/>
-  <xacro:arm_link name="d" m="1" x="0.065" y="0.15" z="0.065"/>
-  <xacro:arm_link name="e" m="1" x="0.15" y="0.155" z="0.032"/>
+  <xacro:arm_link name="d" m="1" x="0.065" y="0.1" z="0.065" dx="-0.0325"/>
+  <xacro:arm_link name="e" m="1" x="0.032" y="0.15" z="0.032" dx="0.05"/>
   <xacro:arm_link name="la_base" m="0.1" x="0.01" y="0.01" z="0.08" dz="0.1"/>
   <xacro:arm_link name="la_piston" m="0.1" x="0.01" y="0.01" z="0.05" dz="-0.05"/>
@@ -290,5 +275,5 @@
     </visual>
     <collision>
-      <origin xyz="0.0875 0 0"/>
+      <origin xyz="0.075 0 0"/>
       <geometry>
         <box size="0.085 0.02 0.03"/>
@@ -364,5 +349,7 @@
   <!-- TODO(quintin): Import the ZED URDF here -->
   <joint name="chassis_link_to_zed_left_camera_frame" type="fixed">
-    <origin xyz="0.3 0 0"/>
+  <!-- Suspension link lengths (measured from blender) -->
+  <!-- TODO: make sure these are real for 2026 -->
+    <origin xyz="0.13 0.025 0.025"/>
     <parent link="chassis_link"/>
     <child link="zed_left_camera_frame"/>
@@ -375,6 +362,6 @@
     </collision>
   </link>
-  <joint name="chassis_link_to_long_range_camera_link" type="fixed">
-    <origin xyz="0.3 0 0"/>
+gg  <joint name="chassis_link_to_long_range_camera_link" type="fixed">
+    <origin xyz="0.13 0.025 0.075"/>
     <parent link="chassis_link"/>
     <child link="long_range_camera_link"/>

Commit message: Update mesh origins

File: urdf/rover/rover.urdf.xacro (robot description, xacro)
@@ -2,5 +2,5 @@
 <robot xmlns:xacro="http://www.ros.org/wiki/xacro" name="rover">
   <!-- Constants -->
-  <xacro:property name="base_width" value="0.59892"/>
+  <xacro:property name="base_width" value="0.59812"/>
   <xacro:property name="base_len" value="0.478"/>
   <xacro:property name="base_height" value="0.183"/>
@@ -169,5 +169,5 @@
       <parent link="${side}_rocker_link"/>
       <child link="front_${side}_wheel_link"/>
-      <origin xyz="0.34781 0.28303 ${reflect * 0.15200}"/>
+      <origin xyz="0.34781 0.28163 ${reflect * 0.15235}"/>
       <axis xyz="0 0 1"/>
       <limit effort="${wheel_torque}" velocity="0"/>
@@ -190,6 +190,5 @@
       <parent link="${side}_rocker_link"/>
       <child link="${side}_lambda_lower_link"/>
-      <!-- TODO: figure out what coordinate frame this is in -->
-      <origin xyz="-0.2773 0.15460 ${reflect * 0.05577}"/>
+      <origin xyz="-0.27730 0.15319 ${reflect * 0.05611}"/>
       <axis xyz="0 0 1"/>
       <limit effort="0" velocity="0"/>
@@ -198,5 +197,5 @@
       <parent link="${side}_rocker_link"/>
       <child link="${side}_lambda_crank_front_link"/>
-      <origin xyz="-0.27730 0.01220 ${reflect * 0.09809}"/>
+      <origin xyz="-0.27730 0.01080 ${reflect * 0.09844}"/>
       <axis xyz="0 0 1"/>
       <limit upper="${pi/2}" lower="-${pi/2}" effort="0" velocity="0"/>
@@ -205,5 +204,5 @@
       <parent link="${side}_rocker_link"/>
       <child link="${side}_lambda_crank_rear_link"/>
-      <origin xyz="-0.27730 0.01220 ${reflect * 0.10760}"/>
+      <origin xyz="-0.27730 0.01080 ${reflect * 0.10795}"/>
       <axis xyz="0 0 1"/>
       <limit upper="${pi/2}" lower="-${pi/2}" effort="0" velocity="0"/>
@@ -282,5 +281,5 @@
   </link>
   <joint name="chassis_link_to_arm_a_link" type="prismatic">
-    <origin xyz="0.0 -0.200235 0.09870"/>
+    <origin xyz="0.0 -0.200235 0.10011"/>
     <parent link="chassis_link"/>
     <child link="arm_a_link"/>
@@ -349,6 +348,4 @@
   <!-- TODO(quintin): Import the ZED URDF here -->
   <joint name="chassis_link_to_zed_left_camera_frame" type="fixed">
-  <!-- Suspension link lengths (measured from blender) -->
-  <!-- TODO: make sure these are real for 2026 -->
     <origin xyz="0.13 0.025 0.025"/>
     <parent link="chassis_link"/>

Commit message: Add simulated diff bar

File: urdf/rover/rover.urdf.xacro (robot description, xacro)
@@ -159,10 +159,26 @@
                                  dy="-0.143526"/>
     </link>
-    <joint name="chassis_link_to_${side}_rocker_link" type="revolute">
+    <link name="${side}_diff_bar_connector_link">
+      <xacro:box_inertia m="0.5" d="0.1" w="0.1" h="0.1"/>
+      <visual>
+        <geometry>
+          <mesh filename="package://mrover/urdf/meshes/rover_diff_bar_connector.fbx"/>
+        </geometry>
+      </visual>
+      <collision>
+        <origin xyz="0 0 -0.04605"/>
+        <geometry>
+          <box size="0.01 0.01 0.05"/>
+        </geometry>
+      </collision>
+    </link>
+    <!-- this link is needed to get a 2 dof rotational joint -->
+    <link name="${side}_diff_bar_connector_x_link"/>
+    <joint name="chassis_link_to_${side}_rocker_link" type="continuous">
       <parent link="chassis_link"/>
       <child link="${side}_rocker_link"/>
       <origin xyz="0.0 ${reflect * (base_width/2)} 0" rpy="${-TAU/4} 0 0"/>
       <axis xyz="0 0 1"/>
-      <limit lower="-0.122173" upper="0.523599" effort="0" velocity="0"/>
+      <limit effort="0" velocity="0"/>
     </joint>
     <joint name="${side}_rocker_link_to_front_${side}_wheel_link" type="continuous">
@@ -199,5 +215,5 @@
       <origin xyz="-0.27730 0.01080 ${reflect * 0.09844}"/>
       <axis xyz="0 0 1"/>
-      <limit upper="${pi/2}" lower="-${pi/2}" effort="0" velocity="0"/>
+      <limit upper="1.2" lower="-1.2" effort="0" velocity="0"/>
     </joint>
     <joint name="${side}_rocker_link_to_${side}_lambda_crank_rear_link" type="revolute">
@@ -206,21 +222,53 @@
       <origin xyz="-0.27730 0.01080 ${reflect * 0.10795}"/>
       <axis xyz="0 0 1"/>
-      <limit upper="${pi/2}" lower="-${pi/2}" effort="0" velocity="0"/>
-    </joint>
-    <joint name="${side}_lambda_lower_link_to_${side}_lambda_front_link" type="continuous">
+      <limit upper="1.2" lower="-1.2" effort="0" velocity="0"/>
+    </joint>
+    <joint name="${side}_lambda_lower_link_to_${side}_lambda_front_link" type="revolute">
       <parent link="${side}_lambda_lower_link"/>
       <child link="${side}_lambda_front_link"/>
       <origin xyz="0.15755 -0.05735 ${reflect * 0.04708}"/>
       <axis xyz="0 0 1"/>
-      <limit effort="0" velocity="0"/>
-    </joint>
-    <joint name="${side}_lambda_lower_link_to_${side}_lambda_rear_link" type="continuous">
+      <limit upper="0.8" lower="-0.8" effort="0" velocity="0"/>
+    </joint>
+    <joint name="${side}_lambda_lower_link_to_${side}_lambda_rear_link" type="revolute">
       <parent link="${side}_lambda_lower_link"/>
       <child link="${side}_lambda_rear_link"/>
       <origin xyz="-0.15755 -0.05735 ${reflect * 0.04708}"/>
       <axis xyz="0 0 1"/>
-      <limit effort="0" velocity="0"/>
-    </joint>
-  </xacro:macro>
+      <limit lower="-0.8" upper="0.8" effort="0" velocity="0"/>
+    </joint>
+    <joint name="diff_bar_link_to_${side}_diff_bar_connector_x_link" type="continuous">
+      <parent link="diff_bar_link"/>
+      <child link="${side}_diff_bar_connector_x_link"/>
+      <origin xyz="-0.01143 ${reflect * 0.35547} 0" rpy="0 0 0"/>
+      <axis xyz="1 0 0"/>
+    </joint>
+    <joint name="${side}_diff_bar_connector_x_link_to_${side}_diff_bar_connector_link" type="continuous">
+      <parent link="${side}_diff_bar_connector_x_link"/>
+      <child link="${side}_diff_bar_connector_link"/>
+      <origin xyz="0 0 0" rpy="0 0 0"/>
+      <axis xyz="0 1 0"/>
+    </joint>
+  </xacro:macro>
+  <link name="diff_bar_link">
+    <xacro:box_inertia m="1" d="0.1" w="0.1" h="0.1"/>
+    <visual>
+      <geometry>
+        <mesh filename="package://mrover/urdf/meshes/rover_diff_bar.fbx"/>
+      </geometry>
+    </visual>
+    <collision>
+      <origin xyz="-0.013 0 0"/>
+      <geometry>
+        <box size="0.03 0.65 0.03"/>
+      </geometry>
+    </collision>
+  </link>
+  <joint name="chassis_link_to_diff_bar_link" type="continuous">
+    <parent link="chassis_link"/>
+    <child link="diff_bar_link"/>
+    <origin xyz="-0.37633 0 -0.00587"/>
+    <axis xyz="1 0 0"/>
+  </joint>
   <!-- Joints/Links -->
   <link name="base_link"/>

Commit message: made finger_cam accurate in sim, arm_controller fixes

File: urdf/rover/rover.urdf.xacro (robot description, xacro)
@@ -293,6 +293,6 @@
   </link>
   <joint name="arm_e_link_to_finger_camera" type="fixed">
-    <origin xyz="0 0 0" rpy="0 0 0"/>
-    <parent link="arm_e_link"/>
+    <origin xyz="0.03713988 0 -0.2" rpy="0 -1.134 0"/>
+    <parent link="arm_d_link"/>
     <child link="finger_camera_frame"/>
   </joint>
