Commit message: squash merge teleop-threejs

File: teleoperation/basestation_gui/frontend/public/urdf/arm/arm.urdf (robot description, URDF)
Before this commit: robot arm, 7 links, 6 joints
Links:
- link a_link: geometry visual mesh filename=../meshes/arm_a_fix.glb
- link arm_gripper_link: geometry visual mesh filename=../meshes/arm_gripper_fix.glb
- link b_link: geometry visual mesh filename=../meshes/arm_b_fix.glb
- link base_link: geometry visual mesh filename=../meshes/rover_chassis.glb
- link c_link: geometry visual mesh filename=../meshes/arm_c_fix.glb
- link d_link: geometry visual mesh filename=../meshes/arm_d_fix.glb
- link e_link: geometry visual mesh filename=../meshes/arm_e_fix.glb

File: urdf/arm/arm.urdf.xacro (robot description, xacro)
@@ -103,14 +103,14 @@
   <link name="base_link">
     <xacro:box_inertia m="3.0" w="${base_len}" h="${base_width}" d="${base_height}"/>
-    <xacro:link-visual fileName="chasis.dae" col="red" r="1" g="1" b="1"/>
+    <xacro:link-visual fileName="chasis.glb" col="red" r="1" g="1" b="1"/>
     <!--    <collision>-->
     <!--        <origin rpy="0 0 0" xyz="0 0 -9.5"/>-->
     <!--        <geometry>-->
-    <!--            <mesh filename="package://robo_impls/urdf/rover.dae"/>-->
+    <!--            <mesh filename="package://robo_impls/urdf/rover.glb"/>-->
     <!--        </geometry>-->
     <!--    </collision> -->
   </link>
   <link name="a_link">
-    <xacro:link-visual fileName="link.a.dae"
+    <xacro:link-visual fileName="link.a.glb"
                        col="white" r="1" g="1" b="1"/>
     <!--    <xacro:link-collision-cylinder radius="3.75" x1="0" y1="0" z1="-1.25" x2="0" y2="0" z2="-3.75"/>-->
@@ -120,17 +120,17 @@
   </link>
   <link name="b_link">
-    <xacro:link-visual fileName="link.b.dae"
+    <xacro:link-visual fileName="link.b.glb"
                        col="orange" r="1" g="0.43" b="0"/>
   </link>
   <link name="c_link">
-    <xacro:link-visual fileName="link.c.dae"
+    <xacro:link-visual fileName="link.c.glb"
                        col="yellow" r="1" g="1" b="0"/>
   </link>
   <link name="d_link">
-    <xacro:link-visual fileName="link.d.dae"
+    <xacro:link-visual fileName="link.d.glb"
                        col="green" r="0.43" g="1" b="0"/>
   </link>
   <link name="e_link">
-    <xacro:link-visual fileName="link.e.dae"
+    <xacro:link-visual fileName="link.e.glb"
                        col="blue" r="0" g="0" b="1"/>
   </link>

File: urdf/zed/zed_macro.urdf.xacro (robot description, xacro)
@@ -66,5 +66,5 @@
                 <origin xyz="${screw_offset_x} 0 0" rpy="0 0 0"/>
                 <geometry>
-                    <mesh filename="package://mrover/urdf/meshes/${model}.dae"/>
+                    <mesh filename="package://mrover/urdf/meshes/${model}.glb"/>
                 </geometry>
                 <material name="${model}_mat"/>
@@ -72,5 +72,5 @@
             <collision>
                 <geometry>
-                    <mesh filename="package://mrover/urdf/meshes/${model}.dae"/>
+                    <mesh filename="package://mrover/urdf/meshes/${model}.glb"/>
                 </geometry>
             </collision>
