Commit message: fk working

File: teleoperation/basestation_gui/frontend/public/urdf/rover/rover.urdf (robot description, URDF)
Before this commit: robot rover, 25 links, 11 joints
Joints:
- joint chassis_to_arm_a: axis 0 -1 0 -> 0 1 0; limit lower=0 upper=40 effort=0 velocity=0 -> lower=-40 upper=0 effort=0 velocity=0

Commit message: full rover urdf in threejs

File: teleoperation/basestation_gui/frontend/public/urdf/rover/rover.urdf (robot description, URDF)
Before this commit: robot rover, 25 links, 11 joints
Links:
- removed link center_gps
- removed link imu
- removed link left_gps
- removed link long_range_camera_link
- removed link right_gps
- removed link zed_left_camera_frame
- link arm_base_link: mass 3.0 -> None
- link back_left_wheel_link: mass 3 -> None; geometry visual mesh filename=../meshes/rover_left_wheel_fix.dae
- link back_right_wheel_link: mass 3 -> None; geometry visual mesh filename=../meshes/rover_right_wheel_fix.dae
- link center_left_wheel_link: mass 3 -> None; geometry visual mesh filename=../meshes/rover_left_wheel_fix.dae
- link center_right_wheel_link: mass 3 -> None; geometry visual mesh filename=../meshes/rover_right_wheel_fix.dae
- link chassis_link: mass 15 -> None; geometry visual mesh filename=../meshes/rover_chassis.dae
- link front_left_wheel_link: mass 3 -> None; geometry visual mesh filename=../meshes/rover_left_wheel_fix.dae
- link front_right_wheel_link: mass 3 -> None; geometry visual mesh filename=../meshes/rover_right_wheel_fix.dae
- link left_bogie_link: mass 3 -> None; geometry visual mesh filename=../meshes/rover_left_bogie_fix.dae
- link left_rocker_link: mass 3 -> None; geometry visual mesh filename=../meshes/rover_left_rocker_fix.dae
- link right_bogie_link: mass 3 -> None; geometry visual mesh filename=../meshes/rover_right_bogie_fix.dae
- link right_rocker_link: mass 3 -> None; geometry visual mesh filename=../meshes/rover_right_rocker_fix.dae
Joints:
- removed joint chassis_link_to_center_gps
- removed joint chassis_link_to_imu
- removed joint chassis_link_to_long_range_camera_link
- removed joint chassis_link_to_right_gps
- removed joint chassis_link_to_zed_left_camera_frame
- added joint chassis_link_to_right_rocker_link: type revolute, parent chassis_link, child right_rocker_link, origin xyz=16.4665 -34.5164 41.3435 rpy=0 0 0, axis 0 1 0, limit lower=-0.122173 upper=0.523599
- added joint chassis_to_left_rocker: type revolute, parent chassis_link, child left_rocker_link, origin xyz=16.4665 34.5164 41.3435 rpy=0 0 0, axis 0 1 0, limit lower=-0.122173 upper=0.523599
- added joint left_bogie_to_center_left_wheel: type continuous, parent left_bogie_link, child center_left_wheel_link, origin xyz=-17.3532 9 -14.7659, axis 0 1 0, limit lower=-10 upper=10
- added joint left_bogie_to_front_left_wheel: type continuous, parent left_bogie_link, child front_left_wheel_link, origin xyz=21.5233 9 -14.7933, axis 0 1 0, limit lower=-10 upper=10
- added joint left_rocker_to_back_left_wheel: type continuous, parent left_rocker_link, child back_left_wheel_link, origin xyz=-41.7094 9 -28.513 , axis 0 1 0, limit lower=-10 upper=10
- added joint left_rocker_to_left_bogie: type revolute, parent left_rocker_link, child left_bogie_link, origin xyz=19.8948 0.0226 -13.8674 rpy=0 0 0, axis 0 1 0, limit lower=-0.349066 upper=0.349066
- added joint right_bogie_link_to_center_right_wheel_link: type continuous, parent right_bogie_link, child center_right_wheel_link, origin xyz=-17.3532 -9 -14.7659 rpy=0 0 0, axis 0 1 0, limit lower=-10 upper=10
- added joint right_bogie_link_to_front_right_wheel_link: type continuous, parent right_bogie_link, child front_right_wheel_link, origin xyz=21.5233 -9 -14.7933 rpy=0 0 0, axis 0 1 0, limit lower=-10 upper=10
- added joint right_rocker_link_to_back_right_wheel_link: type continuous, parent right_rocker_link, child back_right_wheel_link, origin xyz=-41.7094 -9 -28.513 rpy=0 0 0, axis 0 1 0, limit lower=-10 upper=10
- added joint right_rocker_link_to_right_bogie_link: type revolute, parent right_rocker_link, child right_bogie_link, origin xyz=19.8948 0.0226 -13.8674 rpy=0 0 0, axis 0 1 0, limit lower=-0.349066 upper=0.349066
- joint arm_a_to_arm_b: limit lower=-0.7853981875 upper=0 effort=0 velocity=0 -> lower=-0.7853981875 upper=0
- joint arm_b_to_arm_c: limit lower=-0.959931 upper=2.87979 effort=0 velocity=0 -> lower=-0.959931 upper=2.87979
- joint arm_c_to_arm_d: limit lower=-2.35619 upper=2.35619 effort=0 velocity=0 -> lower=-2.35619 upper=2.35619
- joint arm_d_to_arm_e: limit lower=-2.35619 upper=2.35619 effort=0 velocity=0 -> lower=-2.35619 upper=2.35619
- joint chassis_to_arm_a: axis 0 1 0 -> 0 -1 0; limit lower=-40 upper=0 effort=0 velocity=0 -> lower=0 upper=40
- joint gripper_link: limit lower=0 upper=8 effort=0 velocity=0 -> lower=0 upper=8

Commit message: Update rover model in GUI

File: teleoperation/basestation_gui/frontend/public/urdf/rover/rover.urdf (robot description, URDF)
Before this commit: robot rover, 19 links, 16 joints
Links:
- removed link arm_base_link
- removed link left_bogie_link
- removed link right_bogie_link
- added link left_lambda_crank_front_link; visual mesh filename=../meshes/rover_front_lambda_crank.glb
- added link left_lambda_crank_rear_link; visual mesh filename=../meshes/rover_rear_lambda_crank.glb
- added link left_lambda_front_link; visual mesh filename=../meshes/rover_left_lambda_front.glb
- added link left_lambda_lower_link; visual mesh filename=../meshes/rover_left_lambda_lower.glb
- added link left_lambda_rear_link; visual mesh filename=../meshes/rover_left_lambda_rear.glb
- added link right_lambda_crank_front_link; visual mesh filename=../meshes/rover_front_lambda_crank.glb
- added link right_lambda_crank_rear_link; visual mesh filename=../meshes/rover_rear_lambda_crank.glb
- added link right_lambda_front_link; visual mesh filename=../meshes/rover_right_lambda_front.glb
- added link right_lambda_lower_link; visual mesh filename=../meshes/rover_right_lambda_lower.glb
- added link right_lambda_rear_link; visual mesh filename=../meshes/rover_right_lambda_rear.glb
- link arm_a_link: geometry visual mesh filename=../meshes/arm_a.glb
- link arm_b_link: geometry visual mesh filename=../meshes/arm_b.glb
- link arm_c_link: geometry visual mesh filename=../meshes/arm_c.glb
- link arm_d_link: geometry visual mesh filename=../meshes/arm_d.glb
- link arm_e_link: geometry visual mesh filename=../meshes/arm_e.glb
- link arm_gripper_link: geometry visual mesh filename=../meshes/arm_gripper.glb
- link back_left_wheel_link: geometry visual mesh filename=../meshes/rover_left_wheel.glb
- link back_right_wheel_link: geometry visual mesh filename=../meshes/rover_right_wheel.glb
- link center_left_wheel_link: geometry visual mesh filename=../meshes/rover_left_wheel.glb
- link center_right_wheel_link: geometry visual mesh filename=../meshes/rover_right_wheel.glb
- link front_left_wheel_link: geometry visual mesh filename=../meshes/rover_left_wheel.glb
- link front_right_wheel_link: geometry visual mesh filename=../meshes/rover_right_wheel.glb
- link left_rocker_link: geometry visual mesh filename=../meshes/rover_left_rocker.glb
- link right_rocker_link: geometry visual mesh filename=../meshes/rover_right_rocker.glb
Joints:
- removed joint gripper_link
- removed joint left_bogie_to_center_left_wheel
- removed joint left_bogie_to_front_left_wheel
- removed joint left_rocker_to_back_left_wheel
- removed joint left_rocker_to_left_bogie
- removed joint right_bogie_to_center_right_wheel
- removed joint right_bogie_to_front_right_wheel
- removed joint right_rocker_to_back_right_wheel
- removed joint right_rocker_to_right_bogie
- added joint arm_e_to_arm_gripper: type prismatic, parent arm_e_link, child arm_gripper_link, origin xyz=8.375 0 0 rpy=0 0 0, axis 0 1 0, limit lower=0 upper=8.8
- added joint base_link_to_chassis_link: type fixed, parent base_link, child chassis_link, origin xyz=21.18 0.047903 40.225 rpy=0 0 0
- added joint left_lambda_front_to_center_left_wheel: type continuous, parent left_lambda_front_link, child center_left_wheel_link, origin xyz=11.343 9.594 -18.319 rpy=0 0 0, axis 0 1 0
- added joint left_lambda_lower_to_left_lambda_front: type revolute, parent left_lambda_lower_link, child left_lambda_front_link, origin xyz=15.755 4.708 5.735 rpy=0 0 0, axis 0 1 0
- added joint left_lambda_lower_to_left_lambda_rear: type revolute, parent left_lambda_lower_link, child left_lambda_rear_link, origin xyz=-15.755 4.708 5.735 rpy=0 0 0, axis 0 1 0
- added joint left_lambda_rear_to_back_left_wheel: type continuous, parent left_lambda_rear_link, child back_left_wheel_link, origin xyz=-11.343 9.594 -18.319 rpy=0 0 0, axis 0 1 0
- added joint left_rocker_to_front_left_wheel: type continuous, parent left_rocker_link, child front_left_wheel_link, origin xyz=34.781 15.7933 -28.303, axis 0 1 0
- added joint left_rocker_to_left_lambda_crank_front: type revolute, parent left_rocker_link, child left_lambda_crank_front_link, origin xyz=-27.73 10.760 -1.220 rpy=0 0 0, axis 0 1 0
- added joint left_rocker_to_left_lambda_crank_rear: type revolute, parent left_rocker_link, child left_lambda_crank_rear_link, origin xyz=-27.73 9.809 -1.220 rpy=0 0 0, axis 0 1 0
- added joint left_rocker_to_left_lambda_lower: type revolute, parent left_rocker_link, child left_lambda_lower_link, origin xyz=-27.73 5.577 -15.460 rpy=0 0 0, axis 0 1 0
- added joint right_lambda_front_to_center_right_wheel: type continuous, parent right_lambda_front_link, child center_right_wheel_link, origin xyz=11.343 -9.594 -18.319 rpy=0 0 0, axis 0 1 0
- added joint right_lambda_lower_to_right_lambda_front: type revolute, parent right_lambda_lower_link, child right_lambda_front_link, origin xyz=15.755 -4.708 5.735 rpy=0 0 0, axis 0 1 0
- added joint right_lambda_lower_to_right_lambda_rear: type revolute, parent right_lambda_lower_link, child right_lambda_rear_link, origin xyz=-15.755 -4.708 5.735 rpy=0 0 0, axis 0 1 0
- added joint right_lambda_rear_to_back_right_wheel: type continuous, parent right_lambda_rear_link, child back_right_wheel_link, origin xyz=-11.343 -9.594 -18.319 rpy=0 0 0, axis 0 1 0
- added joint right_rocker_to_front_right_wheel: type continuous, parent right_rocker_link, child front_right_wheel_link, origin xyz=34.781 -15.7933 -28.303, axis 0 1 0
- added joint right_rocker_to_right_lambda_crank_front: type revolute, parent right_rocker_link, child right_lambda_crank_front_link, origin xyz=-27.73 -10.760 -1.220 rpy=0 0 0, axis 0 1 0
- added joint right_rocker_to_right_lambda_crank_rear: type revolute, parent right_rocker_link, child right_lambda_crank_rear_link, origin xyz=-27.73 -9.809 -1.220 rpy=0 0 0, axis 0 1 0
- added joint right_rocker_to_right_lambda_lower: type revolute, parent right_rocker_link, child right_lambda_lower_link, origin xyz=-27.73 -5.577 -15.460 rpy=0 0 0, axis 0 1 0
- joint arm_a_to_arm_b: limit lower=-0.7853981875 upper=0 -> lower=-1.344 upper=0.2617; origin xyz=3.4348 -0.0005 4.9028 rpy=0 0 0 -> xyz=4.452 0 5.163 rpy=0 0 0
- joint arm_b_to_arm_c: limit lower=-0.959931 upper=2.87979 -> lower=-1.0471 upper=3.0543; origin xyz=53.4363 0.0005 0.9052 rpy=0 0 0 -> xyz=53.271 0 0 rpy=0 0 0
- joint arm_c_to_arm_d: limit lower=-2.35619 upper=2.35619 -> lower=-1.1344 upper=1.1344; origin xyz=54.6037 0 8.8594 rpy=0 0 0 -> xyz=39.525 0 8.329 rpy=0 0 0
- joint arm_d_to_arm_e: origin xyz=4.488 0 0 rpy=0 0 0 -> xyz=0 0 0 rpy=1.570796 0 0
- joint chassis_to_arm_a: origin xyz=16.4882 20.0235 49.1172 rpy=0 0 0 -> xyz=0 6.5 9.87 rpy=0 0 0
- joint chassis_to_left_rocker: limit lower=-0.122173 upper=0.523599 -> (none); origin xyz=16.4665 34.5164 41.3435 rpy=0 0 0 -> xyz=0 29.946 0 rpy=0 0 0
- joint chassis_to_right_rocker: limit lower=-0.122173 upper=0.523599 -> (none); origin xyz=16.4665 -34.5164 41.3435 rpy=0 0 0 -> xyz=0 -29.946 0 rpy=0 0 0

Commit message: Update rover model in GUI

File: teleoperation/basestation_gui/frontend/public/urdf/rover/rover.urdf (robot description, URDF)
Before this commit: robot rover, 19 links, 16 joints
Links:
- removed link arm_base_link
- removed link left_bogie_link
- removed link right_bogie_link
- added link left_lambda_crank_front_link; visual mesh filename=../meshes/rover_front_lambda_crank.glb
- added link left_lambda_crank_rear_link; visual mesh filename=../meshes/rover_rear_lambda_crank.glb
- added link left_lambda_front_link; visual mesh filename=../meshes/rover_left_lambda_front.glb
- added link left_lambda_lower_link; visual mesh filename=../meshes/rover_left_lambda_lower.glb
- added link left_lambda_rear_link; visual mesh filename=../meshes/rover_left_lambda_rear.glb
- added link right_lambda_crank_front_link; visual mesh filename=../meshes/rover_front_lambda_crank.glb
- added link right_lambda_crank_rear_link; visual mesh filename=../meshes/rover_rear_lambda_crank.glb
- added link right_lambda_front_link; visual mesh filename=../meshes/rover_right_lambda_front.glb
- added link right_lambda_lower_link; visual mesh filename=../meshes/rover_right_lambda_lower.glb
- added link right_lambda_rear_link; visual mesh filename=../meshes/rover_right_lambda_rear.glb
- link arm_a_link: geometry visual mesh filename=../meshes/arm_a.glb
- link arm_b_link: geometry visual mesh filename=../meshes/arm_b.glb
- link arm_c_link: geometry visual mesh filename=../meshes/arm_c.glb
- link arm_d_link: geometry visual mesh filename=../meshes/arm_d.glb
- link arm_e_link: geometry visual mesh filename=../meshes/arm_e.glb
- link arm_gripper_link: geometry visual mesh filename=../meshes/arm_gripper.glb
- link back_left_wheel_link: geometry visual mesh filename=../meshes/rover_left_wheel.glb
- link back_right_wheel_link: geometry visual mesh filename=../meshes/rover_right_wheel.glb
- link center_left_wheel_link: geometry visual mesh filename=../meshes/rover_left_wheel.glb
- link center_right_wheel_link: geometry visual mesh filename=../meshes/rover_right_wheel.glb
- link chassis_link: geometry visual mesh filename=../meshes/rover_chassis.glb
- link front_left_wheel_link: geometry visual mesh filename=../meshes/rover_left_wheel.glb
- link front_right_wheel_link: geometry visual mesh filename=../meshes/rover_right_wheel.glb
- link left_rocker_link: geometry visual mesh filename=../meshes/rover_left_rocker.glb
- link right_rocker_link: geometry visual mesh filename=../meshes/rover_right_rocker.glb
Joints:
- removed joint gripper_link
- removed joint left_bogie_to_center_left_wheel
- removed joint left_bogie_to_front_left_wheel
- removed joint left_rocker_to_back_left_wheel
- removed joint left_rocker_to_left_bogie
- removed joint right_bogie_to_center_right_wheel
- removed joint right_bogie_to_front_right_wheel
- removed joint right_rocker_to_back_right_wheel
- removed joint right_rocker_to_right_bogie
- added joint arm_e_to_arm_gripper: type prismatic, parent arm_e_link, child arm_gripper_link, origin xyz=8.375 0 0 rpy=0 0 0, axis 0 1 0, limit lower=0 upper=8.8
- added joint base_link_to_chassis_link: type fixed, parent base_link, child chassis_link, origin xyz=21.18 0.047903 40.225 rpy=0 0 0
- added joint left_lambda_front_to_center_left_wheel: type continuous, parent left_lambda_front_link, child center_left_wheel_link, origin xyz=11.343 9.594 -18.319 rpy=0 0 0, axis 0 1 0
- added joint left_lambda_lower_to_left_lambda_front: type revolute, parent left_lambda_lower_link, child left_lambda_front_link, origin xyz=15.755 4.708 5.735 rpy=0 0 0, axis 0 1 0
- added joint left_lambda_lower_to_left_lambda_rear: type revolute, parent left_lambda_lower_link, child left_lambda_rear_link, origin xyz=-15.755 4.708 5.735 rpy=0 0 0, axis 0 1 0
- added joint left_lambda_rear_to_back_left_wheel: type continuous, parent left_lambda_rear_link, child back_left_wheel_link, origin xyz=-11.343 9.594 -18.319 rpy=0 0 0, axis 0 1 0
- added joint left_rocker_to_front_left_wheel: type continuous, parent left_rocker_link, child front_left_wheel_link, origin xyz=34.781 15.7933 -28.303, axis 0 1 0
- added joint left_rocker_to_left_lambda_crank_front: type revolute, parent left_rocker_link, child left_lambda_crank_front_link, origin xyz=-27.73 10.760 -1.220 rpy=0 0 0, axis 0 1 0
- added joint left_rocker_to_left_lambda_crank_rear: type revolute, parent left_rocker_link, child left_lambda_crank_rear_link, origin xyz=-27.73 9.809 -1.220 rpy=0 0 0, axis 0 1 0
- added joint left_rocker_to_left_lambda_lower: type revolute, parent left_rocker_link, child left_lambda_lower_link, origin xyz=-27.73 5.577 -15.460 rpy=0 0 0, axis 0 1 0
- added joint right_lambda_front_to_center_right_wheel: type continuous, parent right_lambda_front_link, child center_right_wheel_link, origin xyz=11.343 -9.594 -18.319 rpy=0 0 0, axis 0 1 0
- added joint right_lambda_lower_to_right_lambda_front: type revolute, parent right_lambda_lower_link, child right_lambda_front_link, origin xyz=15.755 -4.708 5.735 rpy=0 0 0, axis 0 1 0
- added joint right_lambda_lower_to_right_lambda_rear: type revolute, parent right_lambda_lower_link, child right_lambda_rear_link, origin xyz=-15.755 -4.708 5.735 rpy=0 0 0, axis 0 1 0
- added joint right_lambda_rear_to_back_right_wheel: type continuous, parent right_lambda_rear_link, child back_right_wheel_link, origin xyz=-11.343 -9.594 -18.319 rpy=0 0 0, axis 0 1 0
- added joint right_rocker_to_front_right_wheel: type continuous, parent right_rocker_link, child front_right_wheel_link, origin xyz=34.781 -15.7933 -28.303, axis 0 1 0
- added joint right_rocker_to_right_lambda_crank_front: type revolute, parent right_rocker_link, child right_lambda_crank_front_link, origin xyz=-27.73 -10.760 -1.220 rpy=0 0 0, axis 0 1 0
- added joint right_rocker_to_right_lambda_crank_rear: type revolute, parent right_rocker_link, child right_lambda_crank_rear_link, origin xyz=-27.73 -9.809 -1.220 rpy=0 0 0, axis 0 1 0
- added joint right_rocker_to_right_lambda_lower: type revolute, parent right_rocker_link, child right_lambda_lower_link, origin xyz=-27.73 -5.577 -15.460 rpy=0 0 0, axis 0 1 0
- joint arm_a_to_arm_b: limit lower=-0.7853981875 upper=0 -> lower=-1.344 upper=0.2617; origin xyz=3.4348 -0.0005 4.9028 rpy=0 0 0 -> xyz=4.452 0 5.163 rpy=0 0 0
- joint arm_b_to_arm_c: limit lower=-0.959931 upper=2.87979 -> lower=-1.0471 upper=3.0543; origin xyz=53.4363 0.0005 0.9052 rpy=0 0 0 -> xyz=53.271 0 0 rpy=0 0 0
- joint arm_c_to_arm_d: limit lower=-2.35619 upper=2.35619 -> lower=-1.1344 upper=1.1344; origin xyz=54.6037 0 8.8594 rpy=0 0 0 -> xyz=39.525 0 8.329 rpy=0 0 0
- joint arm_d_to_arm_e: origin xyz=4.488 0 0 rpy=0 0 0 -> xyz=0 0 0 rpy=1.570796 0 0
- joint chassis_to_arm_a: origin xyz=16.4882 20.0235 49.1172 rpy=0 0 0 -> xyz=0 6.5 9.87 rpy=0 0 0
- joint chassis_to_left_rocker: limit lower=-0.122173 upper=0.523599 -> (none); origin xyz=16.4665 34.5164 41.3435 rpy=0 0 0 -> xyz=0 29.946 0 rpy=0 0 0
- joint chassis_to_right_rocker: limit lower=-0.122173 upper=0.523599 -> (none); origin xyz=16.4665 -34.5164 41.3435 rpy=0 0 0 -> xyz=0 -29.946 0 rpy=0 0 0

Commit message: Fix joint A transform

File: teleoperation/basestation_gui/frontend/public/urdf/rover/rover.urdf (robot description, URDF)
Before this commit: robot rover, 26 links, 25 joints
Joints:
- joint chassis_to_arm_a: origin xyz=0 6.5 9.87 rpy=0 0 0 -> xyz=0 22.5 9.87 rpy=0 0 0
